File: demo-8/PCB/esp32/_autosave-esp32.sch (KiCad schematic (older format))
At the start: 9 parts, among them J1 Conn_01x02_Female, J2 Conn_01x04_Female, J3 Conn_01x04_Female

Commit message: working on pcb
Parts:
- Q1: renamed from Q?; footprint (none) -> Package_SIP:SIP3_11.6x8.5mm
- gave numbers to parts that had none: 1
Other:
- moved on the sheet: R2, R3
Changed lines of the file:
@@
 L Device:R R3
 U 1 1 5F7B8980
-P 7550 3700
-F 0 "R3" V 7757 3700 50  0000 C CNN
-F 1 "10k" V 7666 3700 50  0000 C CNN
-F 2 "Resistor_THT:R_Axial_DIN0204_L3.6mm_D1.6mm_P5.08mm_Horizontal" V 7480 3700 50  0001 C CNN
-F 3 "~" H 7550 3700 50  0001 C CNN
-	1    7550 3700
-	0    -1   -1   0
-$EndComp
-Text GLabel 7400 3700 0    50   Input ~ 0
+P 7550 3650
+F 0 "R3" V 7757 3650 50  0000 C CNN
+F 1 "10k" V 7666 3650 50  0000 C CNN
+F 2 "Resistor_THT:R_Axial_DIN0204_L3.6mm_D1.6mm_P5.08mm_Horizontal" V 7480 3650 50  0001 C CNN
+F 3 "~" H 7550 3650 50  0001 C CNN
+	1    7550 3650
+	0    -1   -1   0
+$EndComp
+Text GLabel 7400 3650 0    50   Input ~ 0
 3.3V
 $Comp
 L Device:R R2
 U 1 1 5F7BF1BF
-P 7500 3500
-F 0 "R2" V 7707 3500 50  0000 C CNN
-F 1 "10k" V 7616 3500 50  0000 C CNN
-F 2 "Resistor_THT:R_Axial_DIN0204_L3.6mm_D1.6mm_P5.08mm_Horizontal" V 7430 3500 50  0001 C CNN
-F 3 "~" H 7500 3500 50  0001 C CNN
-	1    7500 3500
-	0    -1   -1   0
-$EndComp
-Text GLabel 7350 3500 0    50   Input ~ 0
+P 7500 3450
+F 0 "R2" V 7707 3450 50  0000 C CNN
+F 1 "10k" V 7616 3450 50  0000 C CNN
+F 2 "Resistor_THT:R_Axial_DIN0204_L3.6mm_D1.6mm_P5.08mm_Horizontal" V 7430 3450 50  0001 C CNN
+F 3 "~" H 7500 3450 50  0001 C CNN
+	1    7500 3450
+	0    -1   -1   0
+$EndComp
+Text GLabel 7350 3450 0    50   Input ~ 0
 3.3V
 $Comp
@@
 $EndComp
 $Comp
-L Connector:Conn_01x04_Female J?
+L Connector:Conn_01x04_Female J4
 U 1 1 5F7DA04A
 P 8100 2100
-F 0 "J?" H 8128 2076 50  0000 L CNN
+F 0 "J4" H 8128 2076 50  0000 L CNN
 F 1 "Conn_01x04_Female" H 8128 1985 50  0000 L CNN
 F 2 "Connector_PinHeader_1.27mm:PinHeader_1x04_P1.27mm_Vertical" H 8100 2100 50  0001 C CNN
@@
 $EndComp
 $Comp
-L power:GND #PWR?
+L power:GND #PWR0101
 U 1 1 5F7DA7C0
 P 7900 2000
-F 0 "#PWR?" H 7900 1750 50  0001 C CNN
+F 0 "#PWR0101" H 7900 1750 50  0001 C CNN
 F 1 "GND" V 7905 1872 50  0000 R CNN
 F 2 "" H 7900 2000 50  0001 C CNN
@@
 $EndComp
 $Comp
-L power:+1V5 #PWR?
+L power:+1V5 #PWR0102
 U 1 1 5F7DCBD1
 P 7900 2100
-F 0 "#PWR?" H 7900 1950 50  0001 C CNN
+F 0 "#PWR0102" H 7900 1950 50  0001 C CNN
 F 1 "+1V5" V 7915 2228 50  0000 L CNN
 F 2 "" H 7900 2100 50  0001 C CNN
@@
 $EndComp
 $Comp
-L Device:Q_NPN_BCE Q?
+L Device:Q_NPN_BCE Q1
 U 1 1 5F7DE371
 P 7300 2450
-F 0 "Q?" H 7491 2496 50  0000 L CNN
+F 0 "Q1" H 7491 2496 50  0000 L CNN
 F 1 "Q_NPN_BCE" H 7491 2405 50  0000 L CNN
-F 2 "" H 7500 2550 50  0001 C CNN
+F 2 "Package_SIP:SIP3_11.6x8.5mm" H 7500 2550 50  0001 C CNN
 F 3 "~" H 7300 2450 50  0001 C CNN
 	1    7300 2450
@@
 $EndComp
 $Comp
-L power:GND #PWR?
+L power:GND #PWR0103
 U 1 1 5F7E1AA7
 P 7400 2650
-F 0 "#PWR?" H 7400 2400 50  0001 C CNN
+F 0 "#PWR0103" H 7400 2400 50  0001 C CNN
 F 1 "GND" H 7405 2477 50  0000 C CNN
 F 2 "" H 7400 2650 50  0001 C CNN
@@
 Wire Wire Line
 	6100 3550 6100 3350
-Connection ~ 7700 3700
-Wire Wire Line
-	7700 3700 7700 3750
-Wire Wire Line
-	6000 3650 6100 3650
-Wire Wire Line
-	6100 3650 6100 3600
-Wire Wire Line
-	6100 3600 7650 3600
-Wire Wire Line
-	7650 3600 7650 3500
-Wire Wire Line
-	7700 3350 7700 3700
+Wire Wire Line
+	7700 3350 7700 3650
 Wire Wire Line
 	7650 3250 8000 3250
-Connection ~ 7650 3500
-Wire Wire Line
-	7650 3500 7650 3250
 Wire Wire Line
 	7600 3350 7600 3250
@@
 Wire Wire Line
 	7600 3250 7600 3150
+$Comp
+L power:PWR_FLAG #FLG0101
+U 1 1 5F80358D
+P 3800 2550
+F 0 "#FLG0101" H 3800 2625 50  0001 C CNN
+F 1 "PWR_FLAG" H 3800 2723 50  0000 C CNN
+F 2 "" H 3800 2550 50  0001 C CNN
+F 3 "~" H 3800 2550 50  0001 C CNN
+	1    3800 2550
+	-1   0    0    1
+$EndComp
+Connection ~ 3800 2550
+$Comp
+L power:PWR_FLAG #FLG0102
+U 1 1 5F8042DE
+P 3800 2450
+F 0 "#FLG0102" H 3800 2525 50  0001 C CNN
+F 1 "PWR_FLAG" H 3800 2623 50  0000 C CNN
+F 2 "" H 3800 2450 50  0001 C CNN
+F 3 "~" H 3800 2450 50  0001 C CNN
+	1    3800 2450
+	1    0    0    -1
+$EndComp
+Connection ~ 3800 2450
+Wire Wire Line
+	7650 3450 7650 3250
+Wire Wire Line
+	7650 3450 7650 3550
+Wire Wire Line
+	7650 3550 6150 3550
+Wire Wire Line
+	6150 3550 6150 3650
+Connection ~ 7650 3450
+Wire Wire Line
+	6000 3650 6150 3650
+Connection ~ 7700 3650
+Wire Wire Line
+	7700 3650 7700 3750
 $EndSCHEMATC
