File: demo-8/PCB/esp32/esp32.kicad_pcb (KiCad board)
At the start: 2 copper layers, 7 parts, among them J1 Conn_01x02_Female, J2 Conn_01x04_Female, J3 Conn_01x04_Female

Commit message: working on pcb
Parts:
- added J4: Conn_01x04_Female, Connector_PinHeader_1.27mm:PinHeader_1x04_P1.27mm_Vertical, F.Cu at (248.9, 76.2)
- added Q1: Q_NPN_BCE, Package_SIP:SIP3_11.6x8.5mm, F.Cu at (237.3, 81.8)
Connections:
- J2 pad 1: Net-(J2-Pad1) -> +1V5
- R2 pad 1: Net-(J3-Pad3) -> 3.3V
- R2 pad 2: 3.3V -> Net-(J3-Pad3)
Routing:
- net 3.3V: track 88.3 -> 168.2 mm
- net Net-(MD1-Pad23): track 0.00 -> 17.2 mm
- net Net-(J4-Pad3): track 0.00 -> 11.9 mm
