File: demo-11-esphome-module/schematics/hamodule/hamodule.sch (KiCad schematic (older format))
At the start: 26 parts

Commit message: finished v1
Parts:
- removed J?: Conn_01x02_Female, symbol Connector:Conn_01x02_Female
- removed J? (x2): Conn_01x08_Female, symbol Connector:Conn_01x08_Female
- removed PS? (x4): RAC05-05SK, Converter_ACDC:Converter_ACDC_RECOM_RAC05-xxSK_THT, symbol Converter_ACDC:RAC05-05SK
- removed R? (x4): 340, symbol Device:R
- added D2, D3, D4: DIODE, Diode_THT:D_5W_P10.16mm_Horizontal, symbol pspice:DIODE
- added H1, H2, H3, H4, H5, H6, H7, H8: MountingHole_Pad, MountingHole:MountingHole_3.2mm_M3_ISO14580_Pad, symbol Mechanical:MountingHole_Pad
- added J1, J2, J3: 1864053, 1864053:1864053, symbol wire-to-pcb-phoenix:1864053
- added K2, K3, K4: G5Q-1, Relay_THT:Relay_SPDT_Omron-G5Q-1, symbol Relay:G5Q-1
- added Q2, Q3, Q4: 2N2219, Package_TO_SOT_THT:TO-92_Wide, symbol Transistor_BJT:2N2219
- added R10, R11, R12, R2, R3, R4, R9: 10K, Resistor_THT:R_Axial_DIN0204_L3.6mm_D1.6mm_P7.62mm_Horizontal, symbol Device:R
- added R13, R14, R15, R16: 220, Resistor_THT:R_Axial_DIN0204_L3.6mm_D1.6mm_P7.62mm_Horizontal, symbol Device:R
- D1: renamed from D?; footprint (none) -> Diode_THT:D_5W_P10.16mm_Horizontal
- PS5: renamed from PS?; footprint CONV_RAC15-05SK -> RAC15-05SK:CONV_RAC15-05SK
- Q1: renamed from Q?; footprint Package_TO_SOT_THT:TO-39-3 -> Package_TO_SOT_THT:TO-92_Wide
- R1: renamed from R?; footprint (none) -> Resistor_THT:R_Axial_DIN0204_L3.6mm_D1.6mm_P7.62mm_Horizontal
- R5, R6, R7, R8: renamed from R?; value 340 -> 425; footprint (none) -> Resistor_THT:R_Axial_DIN0204_L3.6mm_D1.6mm_P7.62mm_Horizontal
- U1: renamed from U?; footprint MODULE_ESP32-DEVKITC-32D -> esp32-footprint:MODULE_ESP32-DEVKITC-32D
- U2: renamed from U?; footprint DIP16_IL_VIS -> Package_DIP:DIP-16_W7.62mm
- gave numbers to parts that had none: 5
Connections:
- net labels added: Earth, REO1, REO2, REO3, REO4, Sens1, Sens2, Sens3, Sens4
- net labels removed: GPIO, IN
- wire segments 98 -> 109
- no-connect marks 0 -> 34
Other:
- moved on the sheet: D1, K1, PS1, PS2, PS3, PS4, PS5, Q1, R1, U1, U2
