File: demo-11-esphome-module/schematics-v4/main-project/hamodule.sch (KiCad schematic (older format))
At the start: 48 parts, among them J1 1017505, J2 1017505, J4 1017505, K1 G5Q-1, K2 G5Q-1, K3 G5Q-1, K4 G5Q-1, Q1 2N2219, Q2 2N2219, Q3 2N2219, Q4 2N2219, U1 ESP32-DEVKITC-32D

Commit message: using HCPL3700
Parts:
- removed C1, C2, C3, C4: 4.7uF, Capacitor_THT:CP_Radial_D10.0mm_P3.50mm, symbol Device:CP
- added 22uF1, 22uF2, 22uF3, 22uF4: CP_Small, Capacitor_THT:CP_Radial_D6.3mm_P2.50mm, symbol Device:CP_Small
- added H8, H9: MountingHole_Pad, MountingHole:MountingHole_3.2mm_M3_ISO14580_Pad, symbol Mechanical:MountingHole_Pad
- added U2, U3, U4, U5: HCPL3700, HCPL:ON_Semi-CASE_62605_ISSUE_P-0-0-0, symbol HCPL-3700-000:HCPL3700
- J1, J2, J4: footprint 1017505 -> Phoenix_Conn:1017505
- R11, R12: value 10K -> 47k
- R17, R18, R19, R20, R5, R6: value 110k -> 47k
- R7, R8: value 110k -> 10K
Connections:
- net labels added: LightInputs, PowerSupply, Relays
- wire segments 112 -> 104
Other:
- moved on the sheet: D1, D2, D3, D4, J1, J2, J4, K1, K2, K3, K4, PS1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
