File: demo-11-esphome-module/schematics-v4/main-project/hamodule.kicad_pcb (KiCad board)
At the start: 2 copper layers, 56 parts, among them J1 1017505, J2 1017505, J4 1017505, K1 G5Q-1, K2 G5Q-1, K3 G5Q-1, K4 G5Q-1, Q1 2N2219, Q2 2N2219, Q3 2N2219, Q4 2N2219, U1 ESP32-DEVKITC-32D, U2 4N35, U3 4N35, U4 4N35, U5 4N35

Commit message: using HCPL3700
Parts:
- removed C1, C2, C3, C4: 4.7uF, Capacitor_THT:CP_Radial_D10.0mm_P3.50mm
- removed D5, D6, D7, D8: D_Bridge_+-AA, Diode_THT:Diode_Bridge_Round_D8.9mm
- added 22uF1: CP_Small, Capacitor_THT:CP_Radial_D6.3mm_P2.50mm, F.Cu at (148.8, 50.3)
- added 22uF2: CP_Small, Capacitor_THT:CP_Radial_D6.3mm_P2.50mm, F.Cu at (159.8, 50.3)
- added 22uF3: CP_Small, Capacitor_THT:CP_Radial_D6.3mm_P2.50mm, F.Cu at (170.9, 50.3)
- added 22uF4: CP_Small, Capacitor_THT:CP_Radial_D6.3mm_P2.50mm, F.Cu at (182.1, 50.8)
- added H8: MountingHole_Pad, MountingHole:MountingHole_3.2mm_M3_ISO14580_Pad, F.Cu at (146.1, 80.0)
- added H9: MountingHole_Pad, MountingHole:MountingHole_3.2mm_M3_ISO14580_Pad, F.Cu at (182.6, 80.0)
- J1, J2, J4: footprint 1017505:1017505 -> Phoenix_Conn:1017505
- R11, R12: value 10K -> 47k
- R17, R18, R19, R20, R5, R6: value 110k -> 47k
- R7, R8: value 110k -> 10K
- U2, U3, U4, U5: value 4N35 -> HCPL3700; footprint Package_DIP:DIP-6_W7.62mm -> HCPL:ON_Semi-CASE_62605_ISSUE_P-0-0-0
- moved R12 36.0 mm to (173.5, 45.0)
- moved R11 36.0 mm to (162.3, 45.2)
- moved R7 25.5 mm to (144.3, 66.0), turned to 0 degrees
- moved R10 21.1 mm to (177.0, 66.0), turned to 0 degrees
- moved R9 20.5 mm to (166.1, 66.0), turned to 0 degrees
- moved R19 18.6 mm to (165.6, 41.4), turned to 0 degrees
- moved R8 17.9 mm to (155.2, 66.0), turned to 0 degrees
- moved R18 14.7 mm to (154.7, 41.4), turned to 0 degrees
- moved R17 12.1 mm to (184.4, 45.0), turned to 180 degrees
- moved H3 12.1 mm to (100.1, 20.3)
- moved R5 11.2 mm to (143.5, 41.4), turned to 0 degrees
- moved R20 6.93 mm to (176.8, 41.4), turned to 0 degrees
- moved R6 4.88 mm to (151.1, 45.2), turned to 180 degrees
- moved H6 3.42 mm to (182.6, 20.3)
- moved H4 2.54 mm to (59.4, 31.2)
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Connections:
- K1 pad 4: (no net) -> Net-(K1-Pad4)
- K2 pad 4: (no net) -> Net-(K2-Pad4)
- K3 pad 4: (no net) -> Net-(K3-Pad4)
- K4 pad 4: (no net) -> Net-(K4-Pad4)
- PS1 pad 3: (no net) -> Net-(PS1-Pad3)
- R10 pad 1: GPIO35 -> GPIO33
- R11 pad 1: GPIO32 -> Net-(R11-Pad1)
- R11 pad 2: 3.3V+ -> Net-(R11-Pad2)
- R12 pad 1: GPIO33 -> Net-(R12-Pad1)
- R12 pad 2: 3.3V+ -> Net-(R12-Pad2)
- R17 pad 1: Net-(D7-Pad2) -> Net-(R17-Pad1)
- R18 pad 1: Net-(R17-Pad2) -> Sens2
- R18 pad 2: Net-(R18-Pad2) -> Net-(R11-Pad1)
- R19 pad 1: Net-(D8-Pad2) -> Sens3
- R19 pad 2: Net-(R19-Pad2) -> Net-(R12-Pad1)
- R20 pad 1: Net-(R19-Pad2) -> Sens4
- R20 pad 2: Net-(R20-Pad2) -> Net-(R17-Pad1)
- R5 pad 1: Net-(D5-Pad2) -> Sens1
- R7 pad 1: Net-(D6-Pad2) -> GPIO34
- R7 pad 2: Net-(R7-Pad2) -> 3.3V+
- R8 pad 1: Net-(R7-Pad2) -> GPIO35
- R8 pad 2: Net-(R8-Pad2) -> 3.3V+
- R9 pad 1: GPIO34 -> GPIO32
- U1 pad 10: (no net) -> Net-(U1-Pad10)
- U1 pad 11: (no net) -> Net-(U1-Pad11)
- U1 pad 12: (no net) -> Net-(U1-Pad12)
- U1 pad 13: (no net) -> Net-(U1-Pad13)
- U1 pad 14: (no net) -> Net-(U1-Pad14)
- U1 pad 15: (no net) -> Net-(U1-Pad15)
- U1 pad 16: (no net) -> Net-(U1-Pad16)
- U1 pad 17: (no net) -> Net-(U1-Pad17)
- U1 pad 18: (no net) -> Net-(U1-Pad18)
- U1 pad 2: (no net) -> Net-(U1-Pad2)
- U1 pad 21: (no net) -> Net-(U1-Pad21)
- U1 pad 22: (no net) -> Net-(U1-Pad22)
- U1 pad 23: (no net) -> Net-(U1-Pad23)
- U1 pad 24: (no net) -> Net-(U1-Pad24)
- U1 pad 25: (no net) -> Net-(U1-Pad25)
- U1 pad 26: (no net) -> Net-(U1-Pad26)
- U1 pad 27: (no net) -> Net-(U1-Pad27)
- U1 pad 28: (no net) -> Net-(U1-Pad28)
- U1 pad 29: (no net) -> Net-(U1-Pad29)
- U1 pad 3: (no net) -> Net-(U1-Pad3)
- U1 pad 33: (no net) -> Net-(U1-Pad33)
- U1 pad 35: (no net) -> Net-(U1-Pad35)
- U1 pad 36: (no net) -> Net-(U1-Pad36)
- U1 pad 37: (no net) -> Net-(U1-Pad37)
- U1 pad 38: (no net) -> Net-(U1-Pad38)
- U1 pad 4: (no net) -> Net-(U1-Pad4)
- U1 pad 9: (no net) -> Net-(U1-Pad9)
- U2 pad 1: Net-(D5-Pad1) -> 220VAC(N)
- U2 pad 2: Net-(R6-Pad2) -> Net-(22uF1-Pad1)
- U2 pad 3: (no net) -> Net-(22uF1-Pad2)
- U2 pad 4: 5VGND -> Net-(R6-Pad2)
- U2 pad 5: GPIO34 -> 5VGND
- U2 pad 6: (no net) -> GPIO34
- U3 pad 1: Net-(D6-Pad1) -> 220VAC(N)
- U3 pad 2: Net-(R8-Pad2) -> Net-(22uF2-Pad1)
- U3 pad 3: (no net) -> Net-(22uF2-Pad2)
- U3 pad 4: 5VGND -> Net-(R11-Pad2)
- U3 pad 5: GPIO35 -> 5VGND
- U3 pad 6: (no net) -> GPIO35
- U4 pad 1: Net-(D7-Pad1) -> 220VAC(N)
- U4 pad 2: Net-(R18-Pad2) -> Net-(22uF3-Pad1)
- U4 pad 3: (no net) -> Net-(22uF3-Pad2)
- U4 pad 4: 5VGND -> Net-(R12-Pad2)
- U4 pad 5: GPIO32 -> 5VGND
- U4 pad 6: (no net) -> GPIO32
- U5 pad 1: Net-(D8-Pad1) -> 220VAC(N)
- U5 pad 2: Net-(R20-Pad2) -> Net-(22uF4-Pad1)
- U5 pad 3: (no net) -> Net-(22uF4-Pad2)
- U5 pad 4: 5VGND -> Net-(R17-Pad2)
- U5 pad 5: GPIO33 -> 5VGND
- U5 pad 6: (no net) -> GPIO33
Routing:
- net 220VAC(N): track 171.2 -> 205.8 mm
- net 5VGND: track 281.5 -> 252.6 mm
- net 5V+: track 121.5 -> 138.2 mm
- net GPIO34: track 25.9 -> 9.55 mm
- net Net-(D8-Pad1): track 14.8 -> 0.00 mm
- net Net-(D7-Pad1): track 14.8 -> 0.00 mm
- net Net-(D6-Pad1): track 14.8 -> 0.00 mm
- net Net-(D5-Pad1): track 14.8 -> 0.00 mm
- net 3.3V+: track 51.7 -> 65.1 mm
- net GPIO32: track 47.1 -> 34.4 mm
- net GPIO35: track 35.9 -> 23.2 mm
- net GPIO33: track 58.3 -> 46.5 mm
- net Net-(R12-Pad2): track 0.00 -> 10.6 mm
- net Net-(R11-Pad2): track 0.00 -> 10.3 mm
- net Net-(R7-Pad2): track 9.72 -> 0.00 mm
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
Commit message: some changes to schema
Parts:
- moved H8 1.80 mm to (147.3, 78.7)
- moved H9 1.63 mm to (181.6, 78.7)
- moved H6 1.63 mm to (181.6, 21.6)
Routing:
- net 5VGND: track 252.6 -> 274.1 mm
- net REO1: track 23.3 -> 35.3 mm
- net 220VAC(N): track 205.8 -> 215.7 mm
- net REO4: track 29.6 -> 33.0 mm
- net Sens4: track 20.3 -> 23.0 mm
- net Sens1: track 23.1 -> 25.5 mm
- net REO3: track 22.5 -> 20.5 mm
Other:
- board outline added: 165.1 x 67.3 mm
