File: demo-11-esphome-module/schematics-v5/main-project/hamodule.sch (KiCad schematic (older format))
At the start: 41 parts, among them J1 1017505, J2 1017505, J4 1017505, K1 G5Q-1, K2 G5Q-1, K3 G5Q-1, K4 G5Q-1, U1 ESP32-DEVKITC-32D, U2 HCPL3700, U3 HCPL3700, U4 HCPL3700, U5 HCPL3700, U6 ULN2003A

Commit message: schematics v7
Connections:
- no-connect marks 52 -> 50
Changed lines of the file:
@@
 	0    -1   -1   0
 $EndComp
-NoConn ~ 4350 6900
-NoConn ~ 4350 7000
 NoConn ~ 4750 7050
 NoConn ~ 4750 6950
