File: demo-11-esphome-module/schematics-v6/main-project/hamodule.kicad_pcb (KiCad board)
At the start: 2 copper layers, 153.7 x 76.2 mm, 44 parts, among them J1 1017505, J2 1017505, J3 Conn_01x04, J4 Conn_01x02, J5 Conn_01x04, J6 1017505, K1 G5Q-1, K2 G5Q-1, K3 G5Q-1, K4 G5Q-1, U1 ULN2003A, U2 LD1117S33TR_SOT223, U3 HCPL3700, U4 HCPL3700, U5 HCPL3700, U6 HCPL3700

Commit message: schematics v7
Parts:
- J3: value Conn_01x04 -> Conn-ESP-Relays; footprint Connector_Molex:Molex_KK-396_A-41791-0004_1x04_P3.96mm_Vertical -> Connector_JST:JST_XH_B4B-XH-A_1x04_P2.50mm_Vertical
- J4: footprint Connector_Molex:Molex_KK-396_A-41791-0002_1x02_P3.96mm_Vertical -> Connector_JST:JST_XH_B2B-XH-A_1x02_P2.50mm_Vertical
- J5: value Conn_01x04 -> Conn-Esp-Sensors; footprint Connector_Molex:Molex_KK-396_A-41791-0004_1x04_P3.96mm_Vertical -> Connector_JST:JST_XH_B4B-XH-A_1x04_P2.50mm_Vertical
- moved H6 48.8 mm to (171.4, 38.1)
- moved H3 22.5 mm to (171.4, 15.2)
- moved H8 16.6 mm to (120.7, 15.2)
- moved H9 12.5 mm to (101.6, 15.2)
- moved H1 1.80 mm to (168.9, 82.5)
- moved J3 1.80 mm to (83.8, 82.5)
- moved H2 1.80 mm to (96.5, 82.5)
- moved H5 1.27 mm to (108.0, 82.5)
Connections:
- net Net-(J5-Pad1) renamed EspSens4
- net Net-(J5-Pad2) renamed EspSens3
- net Net-(J5-Pad3) renamed EspSens2
- net Net-(J5-Pad4) renamed EspSens1
- 22uF2 pad 1: Net-(22uF2-Pad1) -> (no net)
- 22uF2 pad 2: Net-(22uF2-Pad2) -> (no net)
- R6 pad 2: Net-(R6-Pad2) -> (no net)
Routing:
- net (no net): track 0.00 -> 42.9 mm
- net Net-(R6-Pad2): track 21.3 -> 0.00 mm
- net Net-(22uF2-Pad1): track 10.8 -> 0.00 mm
- net Net-(22uF2-Pad2): track 10.7 -> 0.00 mm
- net EspSens1: track 28.3 -> 32.7 mm
- net EspSens4: track 27.0 -> 23.4 mm
- net EspSens2: track 14.4 -> 17.3 mm
- net Net-(J3-Pad2): track 8.95 -> 10.2 mm
- net Net-(J3-Pad1): track 9.42 -> 10.2 mm
- net Net-(J3-Pad3): track 9.54 -> 10.2 mm
- net EspSens3: track 12.3 -> 11.8 mm
