File: demo-11-esphome-module/schematics-v6/main-project/hamodule.sch (KiCad schematic (older format))
At the start: 44 parts, among them J1 1017505, J2 1017505, J3 Conn_01x04, J4 Conn_01x02, J5 Conn_01x04, J6 1017505, K1 G5Q-1, K2 G5Q-1, K3 G5Q-1, K4 G5Q-1, U1 ULN2003A, U2 LD1117S33TR_SOT223, U3 HCPL3700, U4 HCPL3700, U5 HCPL3700, U6 HCPL3700

Commit message: schematics v7
Parts:
- added D1, D2, D3, D4: LED, LED_THT:LED_D3.0mm, symbol Device:LED
- added J7: Conn-Buttons, Connector_JST:JST_XH_B5B-XH-A_1x05_P2.50mm_Vertical, symbol Connector_Generic:Conn_01x05
- added J8: Conn-LedIndicators, Connector_JST:JST_XH_B4B-XH-A_1x04_P2.50mm_Vertical, symbol Connector_Generic:Conn_01x05
- added R13, R14, R15, R16: 100, Resistor_THT:R_Axial_DIN0207_L6.3mm_D2.5mm_P7.62mm_Horizontal, symbol Device:R
- 22uF1, 22uF2, 22uF3, 22uF4: footprint Capacitor_THT:CP_Radial_D17.0mm_P7.50mm -> Capacitor_THT:CP_Radial_D10.0mm_P5.00mm
- J3: value Conn_01x04 -> Conn-ESP-Relays; footprint Connector_Molex:Molex_KK-396_A-41791-0004_1x04_P3.96mm_Vertical -> Connector_JST:JST_XH_B4B-XH-A_1x04_P2.50mm_Vertical
- J4: footprint Connector_Molex:Molex_KK-396_A-41791-0002_1x02_P3.96mm_Vertical -> Connector_JST:JST_XH_B2B-XH-A_1x02_P2.50mm_Vertical
- J5: value Conn_01x04 -> Conn-Esp-Sensors; footprint Connector_Molex:Molex_KK-396_A-41791-0004_1x04_P3.96mm_Vertical -> Connector_JST:JST_XH_B4B-XH-A_1x04_P2.50mm_Vertical
- R1, R2, R3, R4: value 10K -> 100; footprint Resistor_THT:R_Axial_DIN0204_L3.6mm_D1.6mm_P7.62mm_Horizontal -> Resistor_THT:R_Axial_DIN0207_L6.3mm_D2.5mm_P7.62mm_Horizontal
- R10, R11, R12, R9: footprint Resistor_THT:R_Axial_DIN0516_L15.5mm_D5.0mm_P5.08mm_Vertical -> Resistor_THT:R_Axial_DIN0516_L15.5mm_D5.0mm_P20.32mm_Horizontal
- U2: footprint Package_TO_SOT_THT:TO-218-3_Vertical -> Package_TO_SOT_THT:TO-220-3_Vertical
- U3, U4, U5, U6: footprint HCPL:ON_Semi-CASE_62605_ISSUE_P-0-0-0 -> Package_DIP:DIP-8_W7.62mm_Socket_LongPads
Connections:
- net labels added: EspSens1, EspSens2, EspSens3, EspSens4
- wire segments 66 -> 63
Other:
- moved on the sheet: J5
