File: demo-11-esphome-module/schematics-v11-makesmaller/main-project/_autosave-hamodule.sch (KiCad schematic (older format))
At the start: 67 parts, among them J1 1017505, J10 GND 3.3V, J11 Current Jumper, J2 Conn-ESP-Relays, J3 1017505, J4 Conn-Buttons, J5 Conn_01x02, J6 Conn-Esp-Sensors, J7 Conn-LedIndicators, J8 1017505, J9 Current Jumper, K1 G5Q-1, K2 G5Q-1, K3 G5Q-1, K4 G5Q-1, U1 ULN2003A, U2 LD1117S33TR_SOT223, U3 HCPL3700, U4 HCPL3700, U5 HCPL3700, U6 HCPL3700

Commit message: 2 resistor + jlcpcb
Parts:
- added R11, R13, R15, R17: 39k1w, Resistor_SMD:R_2512_6332Metric_Pad1.52x3.35mm_HandSolder, symbol Device:R
- F2: value F250V -> 7V-100mA
Connections:
- net Sens1: now also R13.1; no longer R14.1
- net Sens2: now also R11.1; no longer R16.1
- net Sens3: now also R15.1; no longer R12.1
- net Sens4: now also R17.1; no longer R10.1
- new net: R13.2, R14.1
- new net: R11.2, R16.1
- new net: R12.1, R15.2
- new net: R10.1, R17.2
Changed lines of the file:
@@
 	1150 2400 1100 2400
 NoConn ~ 550  2450
-Text GLabel 10400 2850 2    50   Input ~ 0
+Text GLabel 10700 2850 2    50   Input ~ 0
 Sens2
-Text GLabel 10400 5850 2    50   Input ~ 0
+Text GLabel 10700 5850 2    50   Input ~ 0
 Sens4
-Text GLabel 10400 3850 2    50   Input ~ 0
+Text GLabel 10700 3850 2    50   Input ~ 0
 Sens1
 $Comp
@@
 Text GLabel 9800 3750 2    50   Input ~ 0
 220VAC(N)
-Text GLabel 10400 4850 2    50   Input ~ 0
+Text GLabel 10700 4850 2    50   Input ~ 0
 Sens3
 NoConn ~ 1800 7600
@@
 P 5650 1900
 F 0 "F2" V 5450 1900 50  0000 C CNN
-F 1 "F250V" V 5550 1900 50  0000 C CNN
+F 1 "7V-100mA" V 5550 1900 50  0000 C CNN
 F 2 "Fuse:Fuse_Littelfuse_372_D8.50mm" V 5580 1900 50  0001 C CNN
 F 3 "~" H 5650 1900 50  0001 C CNN
@@
 	0    1    1    0
 $EndComp
+$Comp
+L Device:R R17
+U 1 1 61799149
+P 10550 5850
+F 0 "R17" V 10343 5850 50  0001 C CNN
+F 1 "39k1w" V 10650 5900 50  0000 C CNN
+F 2 "Resistor_SMD:R_2512_6332Metric_Pad1.52x3.35mm_HandSolder" V 10480 5850 50  0001 C CNN
+F 3 "https://www.distrelec.ch/en/super-high-power-smd-resistor-2512-82kohm-3w-rnd-components-rnd-155sp123wf8202t2e/p/30150189?q=*&pos=1&origPos=3001&origPageSize=50&digitalDataLayerTerm=resistor&track=true" H 10550 5850 50  0001 C CNN
+F 4 "C25723" H 10550 5850 50  0001 C CNN "JLCPCB"
+	1    10550 5850
+	0    1    1    0
+$EndComp
+$Comp
+L Device:R R15
+U 1 1 6179BC18
+P 10550 4850
+F 0 "R15" V 10343 4850 50  0001 C CNN
+F 1 "39k1w" V 10650 4900 50  0000 C CNN
+F 2 "Resistor_SMD:R_2512_6332Metric_Pad1.52x3.35mm_HandSolder" V 10480 4850 50  0001 C CNN
+F 3 "https://www.distrelec.ch/en/super-high-power-smd-resistor-2512-82kohm-3w-rnd-components-rnd-155sp123wf8202t2e/p/30150189?q=*&pos=1&origPos=3001&origPageSize=50&digitalDataLayerTerm=resistor&track=true" H 10550 4850 50  0001 C CNN
+F 4 "C25723" H 10550 4850 50  0001 C CNN "JLCPCB"
+	1    10550 4850
+	0    1    1    0
+$EndComp
+$Comp
+L Device:R R13
+U 1 1 6179E8C9
+P 10550 3850
+F 0 "R13" V 10343 3850 50  0001 C CNN
+F 1 "39k1w" V 10650 3900 50  0000 C CNN
+F 2 "Resistor_SMD:R_2512_6332Metric_Pad1.52x3.35mm_HandSolder" V 10480 3850 50  0001 C CNN
+F 3 "https://www.distrelec.ch/en/super-high-power-smd-resistor-2512-82kohm-3w-rnd-components-rnd-155sp123wf8202t2e/p/30150189?q=*&pos=1&origPos=3001&origPageSize=50&digitalDataLayerTerm=resistor&track=true" H 10550 3850 50  0001 C CNN
+F 4 "C25723" H 10550 3850 50  0001 C CNN "JLCPCB"
+	1    10550 3850
+	0    1    1    0
+$EndComp
+$Comp
+L Device:R R11
+U 1 1 617A141C
+P 10550 2850
+F 0 "R11" V 10343 2850 50  0001 C CNN
+F 1 "39k1w" V 10650 2900 50  0000 C CNN
+F 2 "Resistor_SMD:R_2512_6332Metric_Pad1.52x3.35mm_HandSolder" V 10480 2850 50  0001 C CNN
+F 3 "https://www.distrelec.ch/en/super-high-power-smd-resistor-2512-82kohm-3w-rnd-components-rnd-155sp123wf8202t2e/p/30150189?q=*&pos=1&origPos=3001&origPageSize=50&digitalDataLayerTerm=resistor&track=true" H 10550 2850 50  0001 C CNN
+F 4 "C25723" H 10550 2850 50  0001 C CNN "JLCPCB"
+	1    10550 2850
+	0    1    1    0
+$EndComp
