File: demo-11-esphome-module/schematics-v11-makesmaller/main-project/hamodule.kicad_pcb (KiCad board)
At the start: 2 copper layers, 109.2 x 76.2 mm, 69 parts, among them J1 1017505, J2 Conn-ESP-Relays, J3 1017505, J4 Conn-Buttons, J5 Conn_01x02, J6 Conn-Esp-Sensors, J7 Conn-LedIndicators, J8 1017505, J9 Current Jumper, K1 G5Q-1, K2 G5Q-1, K3 G5Q-1, K4 G5Q-1, U1 ULN2003A, U2 LD1117S33TR_SOT223, U3 HCPL3700, U4 HCPL3700, U5 HCPL3700, U6 HCPL3700

Commit message: notes and reorganizing
Parts:
- added J10: GND 3.3V, Connector_JST:JST_XH_B2B-XH-A_1x02_P2.50mm_Vertical, F.Cu at (147.0, 137.1)
- added J11: Current Jumper, Connector_PinHeader_2.54mm:PinHeader_1x02_P2.54mm_Vertical, F.Cu at (142.0, 138.5)
- 22uF1, 22uF2, 22uF3, 22uF4: value CP_Small -> 22uF
- R1, R2, R3, R4, R5, R6, R7, R8: value 100 -> 62Ω
- R9: renamed from 150Ω; value 100 -> 150Ω
- RV1: value Varistor250v -> 400V
- moved H5 35.1 mm to (112.6, 134.8)
- moved e 2.19 mm to (117.8, 139.4)
- moved 100uF_1 2.10 mm to (123.5, 135.4)
- moved R9 2.10 mm to (117.7, 135.6)
- moved U2 2.10 mm to (131.3, 137.9)
- moved D9 2.10 mm to (117.7, 137.7)
- moved 100uF_2 1.70 mm to (136.7, 135.7)
- moved H1 1.10 mm to (181.3, 70.9)
- moved H3 0.92 mm to (129.2, 77.2)
Connections:
- 100uF_2 pad 1: 3.3V+ -> Net-(100uF_2-Pad1)
- U2 pad 2: 3.3V+ -> Net-(100uF_2-Pad1)
Routing:
- net GND(5V): track 24.9 -> 37.8 mm
- net Net-(100uF_2-Pad1): track 0.00 -> 10.9 mm
- net 3.3V+: track 206.9 -> 198.7 mm
- net 5V+: track 126.4 -> 131.7 mm
- net EspSens1: track 28.1 -> 30.2 mm
- net Net-(F3-Pad2): track 31.0 -> 29.9 mm
Other:
- board text added: "L 230V"
- board text removed: "L 220V"

Commit message: 2 resistor + jlcpcb
Parts:
- added R11: 39k1w, Resistor_SMD:R_2512_6332Metric_Pad1.52x3.35mm_HandSolder, F.Cu at (188.5, 92.0)
- added R13: 39k1w, Resistor_SMD:R_2512_6332Metric_Pad1.52x3.35mm_HandSolder, F.Cu at (193.6, 92.0)
- added R15: 39k1w, Resistor_SMD:R_2512_6332Metric_Pad1.52x3.35mm_HandSolder, F.Cu at (198.7, 92.0)
- added R17: 39k1w, Resistor_SMD:R_2512_6332Metric_Pad1.52x3.35mm_HandSolder, F.Cu at (203.8, 92.0)
- 22uF1, 22uF2, 22uF3, 22uF4: footprint Capacitor_THT:CP_Radial_D5.0mm_P2.00mm -> Capacitor_SMD:C_1206_3216Metric_Pad1.42x1.75mm_HandSolder
- F2: value F250V -> 7V-100mA
- R10, R12, R14, R16: value 82k3w -> 39k1w
- moved F2 54.3 mm to (137.1, 73.1), turned to 0 degrees
- moved REF** 18.9 mm to (180.3, 91.5)
- moved H7 18.2 mm to (181.5, 108.6)
- moved F3 9.53 mm to (188.5, 107.4)
- moved R10 9.53 mm to (203.8, 100.1)
- moved R12 9.53 mm to (198.7, 100.1)
- moved R14 9.53 mm to (193.6, 100.1)
- moved R16 9.53 mm to (188.5, 100.1)
- moved F4 9.53 mm to (193.6, 107.3)
- moved F5 9.53 mm to (198.7, 107.3)
- moved F6 9.53 mm to (203.8, 107.3)
- moved G*** 6.38 mm to (140.3, 82.6)
- moved 22uF1 2.02 mm to (166.7, 115.0)
- moved 22uF4 1.90 mm to (200.8, 115.0)
- moved 22uF2 1.85 mm to (178.0, 115.0)
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Connections:
- R10 pad 1: Sens4 -> Net-(R10-Pad1)
- R12 pad 1: Sens3 -> Net-(R12-Pad1)
- R14 pad 1: Sens1 -> Net-(R13-Pad2)
- R16 pad 1: Sens2 -> Net-(R11-Pad2)
Routing:
- net 220VAC(N): track 65.8 -> 167.1 mm
- net Net-(F2-Pad1): track 135.6 -> 62.8 mm
- net 3.3V+: track 198.7 -> 187.0 mm
- net Net-(F6-Pad2): track 19.2 -> 9.67 mm
- net Net-(F5-Pad2): track 20.1 -> 10.8 mm
- net Net-(F3-Pad2): track 29.9 -> 22.9 mm
- net Sens2: track 21.1 -> 14.2 mm
- net Net-(F4-Pad2): track 23.2 -> 16.9 mm
- net Net-(R13-Pad2): track 0.00 -> 2.13 mm
- net Net-(R12-Pad1): track 0.00 -> 2.13 mm
- net Net-(R11-Pad2): track 0.00 -> 2.13 mm
- net Net-(R10-Pad1): track 0.00 -> 2.13 mm
- net Net-(22uF1-Pad2): track 4.74 -> 2.92 mm
- net Net-(22uF4-Pad1): track 4.61 -> 2.93 mm
- net Net-(22uF2-Pad1): track 4.54 -> 2.99 mm
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Other:
- outline, holes or cut-outs redrawn
- board text removed: "7V-100mA"
- board text removed: "82kΩ3W"

Commit message: adding minimal
Parts:
- added  : , icons:che, F.Cu at (164.4, 136.0)
- 22uF1, 22uF2, 22uF3, 22uF4: footprint Capacitor_SMD:C_1206_3216Metric_Pad1.42x1.75mm_HandSolder -> Capacitor_Tantalum_SMD:CP_EIA-3528-21_Kemet-B_Pad1.50x2.35mm_HandSolder
- R10, R11, R12, R13, R14, R15, R16, R17: value 39k1w -> 39kΩ1w
- moved H7 3.19 mm to (181.8, 105.5)
- moved 22uF3 1.88 mm to (189.5, 114.4)
- moved 22uF1 0.64 mm to (166.7, 114.4)
- moved 22uF2 0.64 mm to (178.0, 114.4)
- moved 22uF4 0.64 mm to (200.8, 114.4)
Connections:
- net D2 renamed EspR2
- net D3 renamed EspR3
- net Net-(D1-Pad2) renamed EspR4
- net Net-(D4-Pad2) renamed EspR1
Routing:
- net Net-(F4-Pad2): track 16.9 -> 18.7 mm
- net Net-(22uF1-Pad1): track 3.07 -> 4.32 mm
- net Net-(22uF4-Pad2): track 3.11 -> 3.80 mm
- net Net-(22uF2-Pad1): track 2.99 -> 3.68 mm
- net Net-(22uF1-Pad2): track 2.92 -> 3.61 mm
- net Net-(22uF2-Pad2): track 3.00 -> 3.70 mm
- net Net-(22uF4-Pad1): track 2.93 -> 3.57 mm
- net Net-(F3-Pad2): track 22.9 -> 22.3 mm
Other:
- outline, holes or cut-outs redrawn
- board text added: "+"
- board text added: "-"
