File: demo-11-esphome-module/schematics-v11-makesmaller/main-project/hamodule.sch (KiCad schematic (older format))
At the start: 65 parts, among them J1 1017505, J2 Conn-ESP-Relays, J3 1017505, J4 Conn-Buttons, J5 Conn_01x02, J6 Conn-Esp-Sensors, J7 Conn-LedIndicators, J8 1017505, J9 Current Jumper, K1 G5Q-1, K2 G5Q-1, K3 G5Q-1, K4 G5Q-1, U1 ULN2003A, U2 LD1117S33TR_SOT223, U3 HCPL3700, U4 HCPL3700, U5 HCPL3700, U6 HCPL3700

Commit message: notes and reorganizing
Parts:
- added J10: GND 3.3V, Connector_JST:JST_XH_B2B-XH-A_1x02_P2.50mm_Vertical, symbol Connector_Generic:Conn_01x02
- added J11: Current Jumper, Connector_PinHeader_2.54mm:PinHeader_1x02_P2.54mm_Vertical, symbol Connector:Conn_01x02_Male
- 22uF1, 22uF2, 22uF3, 22uF4: value CP_Small -> 22uF
- R1, R2, R3, R4, R5, R6, R7, R8: value 62 -> 62Ω
- R9: value 150 -> 150Ω
- RV1: value Varistor250v -> 400V
Connections:
- net 3.3V+: now also J10.2 (Pin_2), J11.1 (Pin_1); no longer 100uF_2.1, U2.2 (VO)
- net GND(5V): now also J10.1 (Pin_1)
- new net: 100uF_2.1, J11.2 (Pin_2), U2.2 (VO)
Other:
- moved on the sheet: J5
Changed lines of the file:
@@
 Text GLabel 4200 2250 0    50   Input ~ 0
 5V+
-Text GLabel 5000 2250 2    50   Input ~ 0
+Text GLabel 5100 2250 2    50   Input ~ 0
 3.3V+
-Text GLabel 6100 2650 2    50   Input ~ 0
+Text GLabel 6450 2750 2    50   Input ~ 0
 5V+
-Text GLabel 6100 2750 2    50   Input ~ 0
+Text GLabel 6450 2850 2    50   Input ~ 0
 GND(5V)
 Wire Notes Line
@@
 P 7100 4300
 F 0 "R1" V 6893 4300 50  0001 C CNN
-F 1 "62" V 7100 4300 50  0000 C CNN
+F 1 "62Ω" V 7100 4300 50  0000 C CNN
 F 2 "Resistor_SMD:R_0805_2012Metric_Pad1.15x1.40mm_HandSolder" V 7030 4300 50  0001 C CNN
 F 3 "https://www.distrelec.ch/en/high-power-thick-film-smd-resistor-0805-62ohm-330mw-rnd-components-rnd-155hp05w3f620jt5e/p/30111853?q=*&pos=2&origPos=1629&origPageSize=50&track=true" H 7100 4300 50  0001 C CNN
@@
 P 7100 4400
 F 0 "R2" V 6893 4400 50  0001 C CNN
-F 1 "62" V 7100 4400 50  0000 C CNN
+F 1 "62Ω" V 7100 4400 50  0000 C CNN
 F 2 "Resistor_SMD:R_0805_2012Metric_Pad1.15x1.40mm_HandSolder" V 7030 4400 50  0001 C CNN
 F 3 "https://www.distrelec.ch/en/high-power-thick-film-smd-resistor-0805-62ohm-330mw-rnd-components-rnd-155hp05w3f620jt5e/p/30111853?q=*&pos=2&origPos=1629&origPageSize=50&track=true" H 7100 4400 50  0001 C CNN
@@
 P 7100 4500
 F 0 "R3" V 6893 4500 50  0001 C CNN
-F 1 "62" V 7100 4500 50  0000 C CNN
+F 1 "62Ω" V 7100 4500 50  0000 C CNN
 F 2 "Resistor_SMD:R_0805_2012Metric_Pad1.15x1.40mm_HandSolder" V 7030 4500 50  0001 C CNN
 F 3 "https://www.distrelec.ch/en/high-power-thick-film-smd-resistor-0805-62ohm-330mw-rnd-components-rnd-155hp05w3f620jt5e/p/30111853?q=*&pos=2&origPos=1629&origPageSize=50&track=true" H 7100 4500 50  0001 C CNN
@@
 P 7100 4600
 F 0 "R4" V 6893 4600 50  0001 C CNN
-F 1 "62" V 7100 4600 50  0000 C CNN
+F 1 "62Ω" V 7100 4600 50  0000 C CNN
 F 2 "Resistor_SMD:R_0805_2012Metric_Pad1.15x1.40mm_HandSolder" V 7030 4600 50  0001 C CNN
 F 3 "https://www.distrelec.ch/en/high-power-thick-film-smd-resistor-0805-62ohm-330mw-rnd-components-rnd-155hp05w3f620jt5e/p/30111853?q=*&pos=2&origPos=1629&origPageSize=50&track=true" H 7100 4600 50  0001 C CNN
@@
 P 8150 3000
 F 0 "R5" H 8000 3050 50  0000 L CNN
-F 1 "62" H 7950 2950 50  0000 L CNN
+F 1 "62Ω" H 7950 2950 50  0000 L CNN
 F 2 "Resistor_SMD:R_0805_2012Metric_Pad1.15x1.40mm_HandSolder" V 8080 3000 50  0001 C CNN
 F 3 "https://www.distrelec.ch/en/high-power-thick-film-smd-resistor-0805-62ohm-330mw-rnd-components-rnd-155hp05w3f620jt5e/p/30111853?q=*&pos=2&origPos=1629&origPageSize=50&track=true" H 8150 3000 50  0001 C CNN
@@
 P 8200 3950
 F 0 "R6" H 8050 4050 50  0000 L CNN
-F 1 "62" H 8000 3950 50  0000 L CNN
+F 1 "62Ω" H 8000 3950 50  0000 L CNN
 F 2 "Resistor_SMD:R_0805_2012Metric_Pad1.15x1.40mm_HandSolder" V 8130 3950 50  0001 C CNN
 F 3 "https://www.distrelec.ch/en/high-power-thick-film-smd-resistor-0805-62ohm-330mw-rnd-components-rnd-155hp05w3f620jt5e/p/30111853?q=*&pos=2&origPos=1629&origPageSize=50&track=true" H 8200 3950 50  0001 C CNN
@@
 P 8200 4950
 F 0 "R7" H 8000 5000 50  0000 L CNN
-F 1 "62" H 7950 4900 50  0000 L CNN
+F 1 "62Ω" H 7950 4900 50  0000 L CNN
 F 2 "Resistor_SMD:R_0805_2012Metric_Pad1.15x1.40mm_HandSolder" V 8130 4950 50  0001 C CNN
 F 3 "https://www.distrelec.ch/en/high-power-thick-film-smd-resistor-0805-62ohm-330mw-rnd-components-rnd-155hp05w3f620jt5e/p/30111853?q=*&pos=2&origPos=1629&origPageSize=50&track=true" H 8200 4950 50  0001 C CNN
@@
 L Connector_Generic:Conn_01x02 J5
 U 1 1 6143ACB7
-P 5900 2750
-F 0 "J5" H 5818 2425 50  0000 C CNN
-F 1 "Conn_01x02" H 5818 2516 50  0000 C CNN
-F 2 "Connector_JST:JST_XH_B2B-XH-A_1x02_P2.50mm_Vertical" H 5900 2750 50  0001 C CNN
-F 3 "~" H 5900 2750 50  0001 C CNN
-	1    5900 2750
+P 6250 2850
+F 0 "J5" H 6168 2525 50  0000 C CNN
+F 1 "Conn_01x02" H 6168 2616 50  0000 C CNN
+F 2 "Connector_JST:JST_XH_B2B-XH-A_1x02_P2.50mm_Vertical" H 6250 2850 50  0001 C CNN
+F 3 "~" H 6250 2850 50  0001 C CNN
+	1    6250 2850
 	-1   0    0    1
 $EndComp
@@
 P 5200 1450
 F 0 "RV1" H 5079 1404 50  0000 R CNN
-F 1 "Varistor250v" H 5079 1495 50  0000 R CNN
+F 1 "400V" H 5079 1495 50  0000 R CNN
 F 2 "Varistor:RV_Disc_D12mm_W4.2mm_P7.5mm" V 5130 1450 50  0001 C CNN
 F 3 "~" H 5200 1450 50  0001 C CNN
@@
 P 10000 5500
 F 0 "22uF4" H 9912 5454 50  0000 R CNN
-F 1 "CP_Small" H 9912 5545 50  0000 R CNN
+F 1 "22uF" H 9912 5545 50  0000 R CNN
 F 2 "Capacitor_THT:CP_Radial_D5.0mm_P2.00mm" H 10000 5500 50  0001 C CNN
 F 3 "~" H 10000 5500 50  0001 C CNN
@@
 P 10000 4500
 F 0 "22uF3" H 9912 4454 50  0000 R CNN
-F 1 "CP_Small" H 9912 4545 50  0000 R CNN
+F 1 "22uF" H 9912 4545 50  0000 R CNN
 F 2 "Capacitor_THT:CP_Radial_D5.0mm_P2.00mm" H 10000 4500 50  0001 C CNN
 F 3 "~" H 10000 4500 50  0001 C CNN
@@
 P 10000 3500
 F 0 "22uF2" H 9912 3454 50  0000 R CNN
-F 1 "CP_Small" H 9912 3545 50  0000 R CNN
+F 1 "22uF" H 9912 3545 50  0000 R CNN
 F 2 "Capacitor_THT:CP_Radial_D5.0mm_P2.00mm" H 10000 3500 50  0001 C CNN
 F 3 "~" H 10000 3500 50  0001 C CNN
@@
 P 10000 2500
 F 0 "22uF1" H 9912 2454 50  0000 R CNN
-F 1 "CP_Small" H 9912 2545 50  0000 R CNN
+F 1 "22uF" H 9912 2545 50  0000 R CNN
 F 2 "Capacitor_THT:CP_Radial_D5.0mm_P2.00mm" H 10000 2500 50  0001 C CNN
 F 3 "~" H 10000 2500 50  0001 C CNN
@@
 P 8200 5950
 F 0 "R8" H 8050 6000 50  0000 L CNN
-F 1 "62" H 8000 5900 50  0000 L CNN
+F 1 "62Ω" H 8000 5900 50  0000 L CNN
 F 2 "Resistor_SMD:R_0805_2012Metric_Pad1.15x1.40mm_HandSolder" V 8130 5950 50  0001 C CNN
 F 3 "https://www.distrelec.ch/en/high-power-thick-film-smd-resistor-0805-62ohm-330mw-rnd-components-rnd-155hp05w3f620jt5e/p/30111853?q=*&pos=2&origPos=1629&origPageSize=50&track=true" H 8200 5950 50  0001 C CNN
@@
 P 7050 1400
 F 0 "R9" V 6843 1400 50  0000 C CNN
-F 1 "150" V 6934 1400 50  0000 C CNN
+F 1 "150Ω" V 6934 1400 50  0000 C CNN
 F 2 "Resistor_SMD:R_0805_2012Metric_Pad1.15x1.40mm_HandSolder" V 6980 1400 50  0001 C CNN
 F 3 "https://www.distrelec.ch/en/high-power-thick-film-smd-resistor-0805-150ohm-330mw-rnd-components-rnd-155hp05w3f1500t5e/p/30111774?q=*&pos=2&origPos=1787&origPageSize=50&track=true" H 7050 1400 50  0001 C CNN
@@
 Wire Wire Line
 	6800 1500 6800 1650
+Text GLabel 6450 2350 2    50   Input ~ 0
+GND(5V)
+$Comp
+L Connector_Generic:Conn_01x02 J10
+U 1 1 61750993
+P 6250 2350
+F 0 "J10" H 6168 2025 50  0000 C CNN
+F 1 "GND 3.3V" H 6168 2116 50  0000 C CNN
+F 2 "Connector_JST:JST_XH_B2B-XH-A_1x02_P2.50mm_Vertical" H 6250 2350 50  0001 C CNN
+F 3 "~" H 6250 2350 50  0001 C CNN
+	1    6250 2350
+	-1   0    0    1
+$EndComp
+Text GLabel 6450 2250 2    50   Input ~ 0
+3.3V+
+$Comp
+L Connector:Conn_01x02_Male J11
+U 1 1 6176729E
+P 5100 2050
+F 0 "J11" V 5050 2000 50  0001 R CNN
+F 1 "Current Jumper" V 5050 2300 50  0000 R CNN
+F 2 "Connector_PinHeader_2.54mm:PinHeader_1x02_P2.54mm_Vertical" H 5100 2050 50  0001 C CNN
+F 3 "~" H 5100 2050 50  0001 C CNN
+	1    5100 2050
+	0    1    1    0
+$EndComp
 $EndSCHEMATC

Commit message: 2 resistor + jlcpcb
Parts:
- added R? (x4): 39k1w, Resistor_SMD:R_2512_6332Metric_Pad1.52x3.35mm_HandSolder, symbol Device:R
- 22uF1, 22uF2, 22uF3, 22uF4: footprint Capacitor_THT:CP_Radial_D5.0mm_P2.00mm -> Capacitor_SMD:C_1206_3216Metric_Pad1.42x1.75mm_HandSolder; JLCPCB (none) -> C12891
- R10, R12, R14, R16: value 82k3w -> 39k1w; JLCPCB (none) -> C25723
Connections:
- net Sens1: now also R?.1; no longer R14.1
- net Sens2: now also R?.1; no longer R16.1
- net Sens3: now also R?.1; no longer R12.1
- net Sens4: now also R?.1; no longer R10.1
- new net: R14.1, R?.2
- new net: R16.1, R?.2
- new net: R12.1, R?.2
- new net: R10.1, R?.2
Changed lines of the file:
@@
 	1150 2400 1100 2400
 NoConn ~ 550  2450
-Text GLabel 10400 2850 2    50   Input ~ 0
+Text GLabel 10700 2850 2    50   Input ~ 0
 Sens2
-Text GLabel 10400 5850 2    50   Input ~ 0
+Text GLabel 10700 5850 2    50   Input ~ 0
 Sens4
-Text GLabel 10400 3850 2    50   Input ~ 0
+Text GLabel 10700 3850 2    50   Input ~ 0
 Sens1
 $Comp
@@
 Text GLabel 9800 3750 2    50   Input ~ 0
 220VAC(N)
-Text GLabel 10400 4850 2    50   Input ~ 0
+Text GLabel 10700 4850 2    50   Input ~ 0
 Sens3
 NoConn ~ 1800 7600
@@
 P 10250 4850
 F 0 "R12" V 10043 4850 50  0001 C CNN
-F 1 "82k3w" V 10350 4850 50  0000 C CNN
+F 1 "39k1w" V 10350 4850 50  0000 C CNN
 F 2 "Resistor_SMD:R_2512_6332Metric_Pad1.52x3.35mm_HandSolder" V 10180 4850 50  0001 C CNN
 F 3 "https://www.distrelec.ch/en/super-high-power-smd-resistor-2512-82kohm-3w-rnd-components-rnd-155sp123wf8202t2e/p/30150189?q=*&pos=1&origPos=3001&origPageSize=50&digitalDataLayerTerm=resistor&track=true" H 10250 4850 50  0001 C CNN
+F 4 "C25723" H 10250 4850 50  0001 C CNN "JLCPCB"
 	1    10250 4850
 	0    1    1    0
@@
 F 0 "22uF4" H 9912 5454 50  0000 R CNN
 F 1 "22uF" H 9912 5545 50  0000 R CNN
-F 2 "Capacitor_THT:CP_Radial_D5.0mm_P2.00mm" H 10000 5500 50  0001 C CNN
-F 3 "~" H 10000 5500 50  0001 C CNN
+F 2 "Capacitor_SMD:C_1206_3216Metric_Pad1.42x1.75mm_HandSolder" H 10000 5500 50  0001 C CNN
+F 3 "https://jlcpcb.com/parts/componentSearch?isSearch=true&searchTxt=22%20uf" H 10000 5500 50  0001 C CNN
+F 4 "C12891" H 10000 5500 50  0001 C CNN "JLCPCB"
 	1    10000 5500
 	-1   0    0    1
@@
 P 10250 5850
 F 0 "R10" V 10043 5850 50  0001 C CNN
-F 1 "82k3w" V 10350 5900 50  0000 C CNN
+F 1 "39k1w" V 10350 5900 50  0000 C CNN
 F 2 "Resistor_SMD:R_2512_6332Metric_Pad1.52x3.35mm_HandSolder" V 10180 5850 50  0001 C CNN
 F 3 "https://www.distrelec.ch/en/super-high-power-smd-resistor-2512-82kohm-3w-rnd-components-rnd-155sp123wf8202t2e/p/30150189?q=*&pos=1&origPos=3001&origPageSize=50&digitalDataLayerTerm=resistor&track=true" H 10250 5850 50  0001 C CNN
+F 4 "C25723" H 10250 5850 50  0001 C CNN "JLCPCB"
 	1    10250 5850
 	0    1    1    0
@@
 F 0 "22uF3" H 9912 4454 50  0000 R CNN
 F 1 "22uF" H 9912 4545 50  0000 R CNN
-F 2 "Capacitor_THT:CP_Radial_D5.0mm_P2.00mm" H 10000 4500 50  0001 C CNN
-F 3 "~" H 10000 4500 50  0001 C CNN
+F 2 "Capacitor_SMD:C_1206_3216Metric_Pad1.42x1.75mm_HandSolder" H 10000 4500 50  0001 C CNN
+F 3 "https://jlcpcb.com/parts/componentSearch?isSearch=true&searchTxt=22%20uf" H 10000 4500 50  0001 C CNN
+F 4 "C12891" H 10000 4500 50  0001 C CNN "JLCPCB"
 	1    10000 4500
 	-1   0    0    1
@@
 F 0 "22uF2" H 9912 3454 50  0000 R CNN
 F 1 "22uF" H 9912 3545 50  0000 R CNN
-F 2 "Capacitor_THT:CP_Radial_D5.0mm_P2.00mm" H 10000 3500 50  0001 C CNN
-F 3 "~" H 10000 3500 50  0001 C CNN
+F 2 "Capacitor_SMD:C_1206_3216Metric_Pad1.42x1.75mm_HandSolder" H 10000 3500 50  0001 C CNN
+F 3 "https://jlcpcb.com/parts/componentSearch?isSearch=true&searchTxt=22%20uf" H 10000 3500 50  0001 C CNN
+F 4 "C12891" H 10000 3500 50  0001 C CNN "JLCPCB"
 	1    10000 3500
 	-1   0    0    1
@@
 P 10250 2850
 F 0 "R16" V 10043 2850 50  0001 C CNN
-F 1 "82k3w" V 10350 2850 50  0000 C CNN
+F 1 "39k1w" V 10350 2850 50  0000 C CNN
 F 2 "Resistor_SMD:R_2512_6332Metric_Pad1.52x3.35mm_HandSolder" V 10180 2850 50  0001 C CNN
 F 3 "https://www.distrelec.ch/en/super-high-power-smd-resistor-2512-82kohm-3w-rnd-components-rnd-155sp123wf8202t2e/p/30150189?q=*&pos=1&origPos=3001&origPageSize=50&digitalDataLayerTerm=resistor&track=true" H 10250 2850 50  0001 C CNN
+F 4 "C25723" V 10250 2850 50  0001 C CNN "JLCPCB"
 	1    10250 2850
 	0    1    1    0
@@
 F 0 "22uF1" H 9912 2454 50  0000 R CNN
 F 1 "22uF" H 9912 2545 50  0000 R CNN
-F 2 "Capacitor_THT:CP_Radial_D5.0mm_P2.00mm" H 10000 2500 50  0001 C CNN
-F 3 "~" H 10000 2500 50  0001 C CNN
+F 2 "Capacitor_SMD:C_1206_3216Metric_Pad1.42x1.75mm_HandSolder" H 10000 2500 50  0001 C CNN
+F 3 "https://jlcpcb.com/parts/componentSearch?isSearch=true&searchTxt=22%20uf" H 10000 2500 50  0001 C CNN
+F 4 "C12891" H 10000 2500 50  0001 C CNN "JLCPCB"
 	1    10000 2500
 	-1   0    0    1
@@
 P 10250 3850
 F 0 "R14" V 10043 3850 50  0001 C CNN
-F 1 "82k3w" V 10350 3850 50  0000 C CNN
+F 1 "39k1w" V 10350 3850 50  0000 C CNN
 F 2 "Resistor_SMD:R_2512_6332Metric_Pad1.52x3.35mm_HandSolder" V 10180 3850 50  0001 C CNN
 F 3 "https://www.distrelec.ch/en/super-high-power-smd-resistor-2512-82kohm-3w-rnd-components-rnd-155sp123wf8202t2e/p/30150189?q=*&pos=1&origPos=3001&origPageSize=50&digitalDataLayerTerm=resistor&track=true" H 10250 3850 50  0001 C CNN
+F 4 "C25723" H 10250 3850 50  0001 C CNN "JLCPCB"
 	1    10250 3850
 	0    1    1    0
@@
 	0    1    1    0
 $EndComp
+$Comp
+L Device:R R?
+U 1 1 61799149
+P 10550 5850
+F 0 "R?" V 10343 5850 50  0001 C CNN
+F 1 "39k1w" V 10650 5900 50  0000 C CNN
+F 2 "Resistor_SMD:R_2512_6332Metric_Pad1.52x3.35mm_HandSolder" V 10480 5850 50  0001 C CNN
+F 3 "https://www.distrelec.ch/en/super-high-power-smd-resistor-2512-82kohm-3w-rnd-components-rnd-155sp123wf8202t2e/p/30150189?q=*&pos=1&origPos=3001&origPageSize=50&digitalDataLayerTerm=resistor&track=true" H 10550 5850 50  0001 C CNN
+F 4 "C25723" H 10550 5850 50  0001 C CNN "JLCPCB"
+	1    10550 5850
+	0    1    1    0
+$EndComp
+$Comp
+L Device:R R?
+U 1 1 6179BC18
+P 10550 4850
+F 0 "R?" V 10343 4850 50  0001 C CNN
+F 1 "39k1w" V 10650 4900 50  0000 C CNN
+F 2 "Resistor_SMD:R_2512_6332Metric_Pad1.52x3.35mm_HandSolder" V 10480 4850 50  0001 C CNN
+F 3 "https://www.distrelec.ch/en/super-high-power-smd-resistor-2512-82kohm-3w-rnd-components-rnd-155sp123wf8202t2e/p/30150189?q=*&pos=1&origPos=3001&origPageSize=50&digitalDataLayerTerm=resistor&track=true" H 10550 4850 50  0001 C CNN
+F 4 "C25723" H 10550 4850 50  0001 C CNN "JLCPCB"
+	1    10550 4850
+	0    1    1    0
+$EndComp
+$Comp
+L Device:R R?
+U 1 1 6179E8C9
+P 10550 3850
+F 0 "R?" V 10343 3850 50  0001 C CNN
+F 1 "39k1w" V 10650 3900 50  0000 C CNN
+F 2 "Resistor_SMD:R_2512_6332Metric_Pad1.52x3.35mm_HandSolder" V 10480 3850 50  0001 C CNN
+F 3 "https://www.distrelec.ch/en/super-high-power-smd-resistor-2512-82kohm-3w-rnd-components-rnd-155sp123wf8202t2e/p/30150189?q=*&pos=1&origPos=3001&origPageSize=50&digitalDataLayerTerm=resistor&track=true" H 10550 3850 50  0001 C CNN
+F 4 "C25723" H 10550 3850 50  0001 C CNN "JLCPCB"
+	1    10550 3850
+	0    1    1    0
+$EndComp
+$Comp
+L Device:R R?
+U 1 1 617A141C
+P 10550 2850
+F 0 "R?" V 10343 2850 50  0001 C CNN
+F 1 "39k1w" V 10650 2900 50  0000 C CNN
+F 2 "Resistor_SMD:R_2512_6332Metric_Pad1.52x3.35mm_HandSolder" V 10480 2850 50  0001 C CNN
+F 3 "https://www.distrelec.ch/en/super-high-power-smd-resistor-2512-82kohm-3w-rnd-components-rnd-155sp123wf8202t2e/p/30150189?q=*&pos=1&origPos=3001&origPageSize=50&digitalDataLayerTerm=resistor&track=true" H 10550 2850 50  0001 C CNN
+F 4 "C25723" H 10550 2850 50  0001 C CNN "JLCPCB"
+	1    10550 2850
+	0    1    1    0
+$EndComp

Commit message: adding minimal
Parts:
- 22uF1, 22uF2, 22uF3, 22uF4: footprint Capacitor_SMD:C_1206_3216Metric_Pad1.42x1.75mm_HandSolder -> Capacitor_Tantalum_SMD:CP_EIA-3528-21_Kemet-B_Pad1.50x2.35mm_HandSolder; JLCPCB C12891 -> C110051
- C1, C2, C3, C4: JLCPCB (none) -> C235777
- F2: value F250V -> 7V-100mA
- R10, R12, R14, R16: value 39k1w -> 39kΩ1w
- R11, R13, R15, R17: renamed from R?; value 39k1w -> 39kΩ1w
Connections:
- net EspR1: now reaches D4.2 (A), J2.1 (Pin_1)
- net EspR4: now reaches D1.2 (A), J2.4 (Pin_4)
- net D2 renamed EspR2
- net D3 renamed EspR3
Other:
- moved on the sheet: 22uF1, C1, D5, F3, J2, J4, J6, J7, R5, U3
