File: demo-11-esphome-module/schematics-v12-minimal/main-project/hamodule.sch (KiCad schematic (older format))
At the start: 55 parts, among them J1 1017505, J10 GND 3.3V, J11 Current Jumper, J2 ESP Relays, J3 1017505, J5 Conn_01x02, J6 ESP Sensors, J8 1017505, J9 Current Jumper, K1 G5Q-1, K2 G5Q-1, K3 G5Q-1, K4 G5Q-1, U1 ULN2003A, U2 LD1117S33TR_SOT223, U3 HCPL3700, U4 HCPL3700, U5 HCPL3700, U6 HCPL3700

Commit message: gebert + bom
Parts:
- D9: JLCPCB (none) -> C2297
- F3, F4, F5, F6: JLCPCB (none) -> C207063
- R9: JLCPCB (none) -> C17471
Changed lines of the file:
@@
 F 2 "Fuse:Fuse_1812_4532Metric_Pad1.30x3.40mm_HandSolder" V 9880 2650 50  0001 C CNN
 F 3 "https://www.distrelec.ch/en/resettable-smd-fuse-60v-400ma-bel-fuse-0zcg0020af2c/p/30127324?q=fuse+smd&pos=4&origPos=112&origPageSize=50&track=true" H 9950 2650 50  0001 C CNN
+F 4 "C207063" H 9950 2650 50  0001 C CNN "JLCPCB"
 	1    9950 2650
 	0    1    1    0
@@
 F 2 "Fuse:Fuse_1812_4532Metric_Pad1.30x3.40mm_HandSolder" V 9880 3850 50  0001 C CNN
 F 3 "https://www.distrelec.ch/en/resettable-smd-fuse-60v-400ma-bel-fuse-0zcg0020af2c/p/30127324?q=fuse+smd&pos=4&origPos=112&origPageSize=50&track=true" H 9950 3850 50  0001 C CNN
+F 4 "C207063" H 9950 3850 50  0001 C CNN "JLCPCB"
 	1    9950 3850
 	0    1    1    0
@@
 F 2 "Fuse:Fuse_1812_4532Metric_Pad1.30x3.40mm_HandSolder" V 9880 5850 50  0001 C CNN
 F 3 "https://www.distrelec.ch/en/resettable-smd-fuse-60v-400ma-bel-fuse-0zcg0020af2c/p/30127324?q=fuse+smd&pos=4&origPos=112&origPageSize=50&track=true" H 9950 5850 50  0001 C CNN
+F 4 "C207063" H 9950 5850 50  0001 C CNN "JLCPCB"
 	1    9950 5850
 	0    1    1    0
@@
 F 2 "Fuse:Fuse_1812_4532Metric_Pad1.30x3.40mm_HandSolder" V 9880 4850 50  0001 C CNN
 F 3 "https://www.distrelec.ch/en/resettable-smd-fuse-60v-400ma-bel-fuse-0zcg0020af2c/p/30127324?q=fuse+smd&pos=4&origPos=112&origPageSize=50&track=true" H 9950 4850 50  0001 C CNN
+F 4 "C207063" H 9950 4850 50  0001 C CNN "JLCPCB"
 	1    9950 4850
 	0    1    1    0
@@
 F 2 "Resistor_SMD:R_0805_2012Metric_Pad1.15x1.40mm_HandSolder" V 6980 1400 50  0001 C CNN
 F 3 "https://www.distrelec.ch/en/high-power-thick-film-smd-resistor-0805-150ohm-330mw-rnd-components-rnd-155hp05w3f1500t5e/p/30111774?q=*&pos=2&origPos=1787&origPageSize=50&track=true" H 7050 1400 50  0001 C CNN
+F 4 "C17471" H 7050 1400 50  0001 C CNN "JLCPCB"
 	1    7050 1400
 	0    1    1    0
@@
 F 2 "LED_SMD:LED_0805_2012Metric_Pad1.15x1.40mm_HandSolder" H 7050 1500 50  0001 C CNN
 F 3 "https://www.distrelec.ch/en/smd-led-green-575nm-20ma-2v-140-everlight-electronics-17-21sygc-s530-e1-tr8/p/17531205?q=*&pos=9&origPos=371&origPageSize=50&track=true" H 7050 1500 50  0001 C CNN
+F 4 "C2297" H 7050 1500 50  0001 C CNN "JLCPCB"
 	1    7050 1500
 	1    0    0    -1

Commit message: adding caps here and there
Parts:
- added C6, C7: 0.1uF, Capacitor_SMD:C_0805_2012Metric_Pad1.15x1.40mm_HandSolder, symbol Device:CP
- F2: value 7V-100mA -> 250v-40mA
Connections:
- net 5V+: now also C6.1, C7.1
- net GND(5V): now also C5.2, C6.2, C7.2; no longer C5.1
- net at 100uF_2.1, J11.2 (Pin_2), U2.2 (VO): now also C5.1; no longer C5.2
Changed lines of the file:
@@
 NoConn ~ 4100 1400
 NoConn ~ 4100 1500
-Text GLabel 4200 2250 0    50   Input ~ 0
+Text GLabel 4250 2500 0    50   Input ~ 0
 5V+
-Text GLabel 5300 2250 2    50   Input ~ 0
+Text GLabel 5650 2500 2    50   Input ~ 0
 3.3V+
 Text GLabel 6450 2750 2    50   Input ~ 0
@@
 Wire Notes Line
 	7700 6300 11000 6300
-Text GLabel 4600 2650 3    50   Input ~ 0
+Text GLabel 4350 2900 0    50   Input ~ 0
 GND(5V)
 Wire Notes Line
@@
 	4900 1600 4900 1900
 NoConn ~ 1200 7600
-Connection ~ 4950 2250
-Wire Wire Line
-	4950 2250 4900 2250
-Wire Wire Line
-	4600 2550 4600 2650
-Wire Wire Line
-	4250 2550 4250 2650
-Wire Wire Line
-	4250 2650 4600 2650
-Wire Wire Line
-	4600 2650 4950 2650
-Wire Wire Line
-	4950 2650 4950 2550
-Connection ~ 4600 2650
-Wire Wire Line
-	4950 2350 4950 2250
-Wire Wire Line
-	4200 2250 4250 2250
-Wire Wire Line
-	4250 2350 4250 2250
-Connection ~ 4250 2250
-Wire Wire Line
-	4250 2250 4300 2250
+Connection ~ 5300 2500
+Wire Wire Line
+	5300 2500 5250 2500
+Wire Wire Line
+	4950 2800 4950 2900
+Wire Wire Line
+	4600 2900 4950 2900
+Wire Wire Line
+	4950 2900 5300 2900
+Connection ~ 4950 2900
+Wire Wire Line
+	5300 2600 5300 2500
 Text GLabel 9800 3750 2    50   Input ~ 0
 220VAC(N)
@@
 L Device:CP 100uF_2
 U 1 1 615251C7
-P 4950 2500
-F 0 "100uF_2" H 5068 2546 50  0001 L CNN
-F 1 "100uF" H 4650 2500 50  0000 L CNN
-F 2 "Capacitor_THT:CP_Radial_D6.3mm_P2.50mm" H 4988 2350 50  0001 C CNN
-F 3 "~" H 4950 2500 50  0001 C CNN
-	1    4950 2500
+P 5300 2750
+F 0 "100uF_2" H 5418 2796 50  0001 L CNN
+F 1 "100uF" H 5000 2750 50  0000 L CNN
+F 2 "Capacitor_THT:CP_Radial_D6.3mm_P2.50mm" H 5338 2600 50  0001 C CNN
+F 3 "~" H 5300 2750 50  0001 C CNN
+	1    5300 2750
 	1    0    0    -1
 $EndComp
@@
 L Regulator_Linear:LD1117S33TR_SOT223 U2
 U 1 1 61434446
-P 4600 2250
-F 0 "U2" H 4600 2492 50  0001 C CNN
-F 1 "LD1117S33TR_SOT223" H 4600 2401 50  0000 C CNN
-F 2 "Package_TO_SOT_THT:TO-220-3_Vertical" H 4600 2450 50  0001 C CNN
-F 3 "http://www.st.com/st-web-ui/static/active/en/resource/technical/document/datasheet/CD00000544.pdf" H 4700 2000 50  0001 C CNN
-	1    4600 2250
+P 4950 2500
+F 0 "U2" H 4950 2742 50  0001 C CNN
+F 1 "LD1117S33TR_SOT223" H 4950 2651 50  0000 C CNN
+F 2 "Package_TO_SOT_THT:TO-220-3_Vertical" H 4950 2700 50  0001 C CNN
+F 3 "http://www.st.com/st-web-ui/static/active/en/resource/technical/document/datasheet/CD00000544.pdf" H 5050 2250 50  0001 C CNN
+	1    4950 2500
 	1    0    0    -1
 $EndComp
@@
 L Device:CP 100uF_1
 U 1 1 6151DFD1
-P 4250 2500
-F 0 "100uF_1" H 4368 2546 50  0001 L CNN
-F 1 "100uF" H 3900 2500 50  0000 L CNN
-F 2 "Capacitor_THT:CP_Radial_D6.3mm_P2.50mm" H 4288 2350 50  0001 C CNN
-F 3 "~" H 4250 2500 50  0001 C CNN
-	1    4250 2500
+P 4350 2750
+F 0 "100uF_1" H 4468 2796 50  0001 L CNN
+F 1 "100uF" H 4000 2750 50  0000 L CNN
+F 2 "Capacitor_THT:CP_Radial_D6.3mm_P2.50mm" H 4388 2600 50  0001 C CNN
+F 3 "~" H 4350 2750 50  0001 C CNN
+	1    4350 2750
 	1    0    0    -1
 $EndComp
@@
 L Connector:Conn_01x02_Male J11
 U 1 1 6176729E
-P 5300 2050
-F 0 "J11" V 5250 2000 50  0001 R CNN
-F 1 "Current Jumper" V 5250 2300 50  0000 R CNN
-F 2 "Connector_PinHeader_2.54mm:PinHeader_1x02_P2.54mm_Vertical" H 5300 2050 50  0001 C CNN
-F 3 "~" H 5300 2050 50  0001 C CNN
-	1    5300 2050
+P 5650 2300
+F 0 "J11" V 5600 2250 50  0001 R CNN
+F 1 "Current Jumper" V 5600 2550 50  0000 R CNN
+F 2 "Connector_PinHeader_2.54mm:PinHeader_1x02_P2.54mm_Vertical" H 5650 2300 50  0001 C CNN
+F 3 "~" H 5650 2300 50  0001 C CNN
+	1    5650 2300
 	0    1    1    0
 $EndComp
@@
 P 5650 1900
 F 0 "F2" V 5450 1900 50  0000 C CNN
-F 1 "7V-100mA" V 5550 1900 50  0000 C CNN
+F 1 "250v-40mA" V 5550 1900 50  0000 C CNN
 F 2 "Fuse:Fuse_Littelfuse_372_D8.50mm" V 5580 1900 50  0001 C CNN
 F 3 "~" H 5650 1900 50  0001 C CNN
@@
 L power:PWR_FLAG #FLG0108
 U 1 1 619A4871
-P 5300 2250
-F 0 "#FLG0108" H 5300 2325 50  0001 C CNN
-F 1 "PWR_FLAG" H 5300 2423 50  0001 C CNN
-F 2 "" H 5300 2250 50  0001 C CNN
-F 3 "~" H 5300 2250 50  0001 C CNN
-	1    5300 2250
+P 5650 2500
+F 0 "#FLG0108" H 5650 2575 50  0001 C CNN
+F 1 "PWR_FLAG" H 5650 2673 50  0001 C CNN
+F 2 "" H 5650 2500 50  0001 C CNN
+F 3 "~" H 5650 2500 50  0001 C CNN
+	1    5650 2500
 	-1   0    0    1
 $EndComp
@@
 L Device:CP C5
 U 1 1 619D049D
-P 5200 2500
-F 0 "C5" H 5318 2546 50  0001 L CNN
-F 1 "0.1uF" H 5050 2500 50  0000 R CNN
-F 2 "Capacitor_SMD:C_0805_2012Metric_Pad1.15x1.40mm_HandSolder" H 5238 2350 50  0001 C CNN
-F 3 "https://www.distrelec.ch/en/ceramic-capacitor-100nf-50vdc-0805-rnd-components-rnd-1500805b104j500nt/p/30086635?q=smd+capacitor+&pos=5&origPos=990&origPageSize=50&track=true" H 5200 2500 50  0001 C CNN
-F 4 "C235777" H 5200 2500 50  0001 C CNN "JLCPCB"
-	1    5200 2500
-	-1   0    0    1
-$EndComp
-Wire Wire Line
-	4950 2250 5200 2250
-Wire Wire Line
-	5200 2250 5200 2350
-Connection ~ 5200 2250
-Wire Wire Line
-	5200 2650 4950 2650
-Connection ~ 4950 2650
+P 5550 2750
+F 0 "C5" H 5668 2796 50  0001 L CNN
+F 1 "0.1uF" H 5850 2750 50  0000 R CNN
+F 2 "Capacitor_SMD:C_0805_2012Metric_Pad1.15x1.40mm_HandSolder" H 5588 2600 50  0001 C CNN
+F 3 "https://www.distrelec.ch/en/ceramic-capacitor-100nf-50vdc-0805-rnd-components-rnd-1500805b104j500nt/p/30086635?q=smd+capacitor+&pos=5&origPos=990&origPageSize=50&track=true" H 5550 2750 50  0001 C CNN
+F 4 "C235777" H 5550 2750 50  0001 C CNN "JLCPCB"
+	1    5550 2750
+	1    0    0    -1
+$EndComp
+Wire Wire Line
+	5300 2500 5550 2500
+Wire Wire Line
+	5550 2500 5550 2600
+Connection ~ 5550 2500
+Wire Wire Line
+	5550 2900 5300 2900
+Connection ~ 5300 2900
+$Comp
+L Device:CP C7
+U 1 1 61809E87
+P 4600 2750
+F 0 "C7" H 4718 2796 50  0001 L CNN
+F 1 "0.1uF" H 4900 2750 50  0000 R CNN
+F 2 "Capacitor_SMD:C_0805_2012Metric_Pad1.15x1.40mm_HandSolder" H 4638 2600 50  0001 C CNN
+F 3 "https://www.distrelec.ch/en/ceramic-capacitor-100nf-50vdc-0805-rnd-components-rnd-1500805b104j500nt/p/30086635?q=smd+capacitor+&pos=5&origPos=990&origPageSize=50&track=true" H 4600 2750 50  0001 C CNN
+F 4 "C235777" H 4600 2750 50  0001 C CNN "JLCPCB"
+	1    4600 2750
+	1    0    0    -1
+$EndComp
+Wire Wire Line
+	4350 2600 4350 2500
+Wire Wire Line
+	4350 2500 4250 2500
+Wire Wire Line
+	4350 2500 4600 2500
+Connection ~ 4350 2500
+Wire Wire Line
+	4600 2600 4600 2500
+Connection ~ 4600 2500
+Wire Wire Line
+	4600 2500 4650 2500
+Wire Wire Line
+	4600 2900 4350 2900
+Connection ~ 4600 2900
+$Comp
+L Device:CP C6
+U 1 1 6181C340
+P 3950 3950
+F 0 "C6" H 4068 3996 50  0001 L CNN
+F 1 "0.1uF" H 4250 3950 50  0000 R CNN
+F 2 "Capacitor_SMD:C_0805_2012Metric_Pad1.15x1.40mm_HandSolder" H 3988 3800 50  0001 C CNN
+F 3 "https://www.distrelec.ch/en/ceramic-capacitor-100nf-50vdc-0805-rnd-components-rnd-1500805b104j500nt/p/30086635?q=smd+capacitor+&pos=5&origPos=990&origPageSize=50&track=true" H 3950 3950 50  0001 C CNN
+F 4 "C235777" H 3950 3950 50  0001 C CNN "JLCPCB"
+	1    3950 3950
+	0    -1   -1   0
+$EndComp
+Wire Wire Line
+	4350 4000 4100 4000
+Wire Wire Line
+	4100 4000 4100 3950
+Wire Wire Line
+	3800 3950 3650 3950
+Wire Wire Line
+	3650 3950 3650 4900
+Wire Wire Line
+	3650 4900 3950 4900
+Wire Wire Line
+	3950 4900 3950 5000
 $EndSCHEMATC
