File: demo-11-esphome-module/schematics-v13-new-relays/main-project/hamodule.kicad_pcb (KiCad board)
At the start: 2 copper layers, 74.9 x 84.3 mm, 60 parts, among them J1 1017505, J10 GND 3.3V, J11 Current Jumper, J2 ESP Relays, J3 1017505, J5 Conn_01x02, J6 ESP Sensors, J8 1017505, J9 Current Jumper, K1 PCN-124D3MHZ,000, K2 PCN-124D3MHZ,000, K3 PCN-124D3MHZ,000, K4 PCN-124D3MHZ,000, U1 ULN2003A, U2 LD1117S33TR_SOT223, U3 HCPL3700, U4 HCPL3700, U5 HCPL3700, U6 HCPL3700

Commit message: cleaning tags
Parts:
- removed F3, F4, F5, F6: Fuse, Fuse:Fuse_1210_3225Metric_Pad1.42x2.65mm_HandSolder
- K1, K2, K3, K4: value PCN-124D3MHZ,000 -> PCN-105D
- R10, R11, R12, R13, R14, R15, R16, R17: value 39kΩ1w -> 39kΩ3w
- moved H3 107.3 mm to (196.0, 117.7)
- moved H1 91.2 mm to (147.3, 99.4)
- moved H2 27.8 mm to (196.0, 146.1)
- moved G*** 8.03 mm to (189.4, 146.6)
- moved F1 5.34 mm to (140.7, 89.7)
- moved G*** 2.34 mm to (185.4, 117.7)
Connections:
- R10 pad 2: Net-(F6-Pad1) -> Net-(R10-Pad2)
- R12 pad 2: Net-(F5-Pad1) -> Net-(R12-Pad2)
- R14 pad 2: Net-(F4-Pad1) -> Net-(R14-Pad2)
- R16 pad 2: Net-(F3-Pad1) -> Net-(R16-Pad2)
- U3 pad 1: Net-(F3-Pad2) -> Net-(R16-Pad2)
- U4 pad 1: Net-(F4-Pad2) -> Net-(R14-Pad2)
- U5 pad 1: Net-(F5-Pad2) -> Net-(R12-Pad2)
- U6 pad 1: Net-(F6-Pad2) -> Net-(R10-Pad2)
Routing:
- net Net-(R16-Pad2): track 0.00 -> 54.3 mm
- net Net-(F3-Pad2): track 48.5 -> 0.00 mm
- net Net-(R14-Pad2): track 0.00 -> 44.1 mm
- net Net-(F4-Pad2): track 38.3 -> 0.00 mm
- net Net-(R10-Pad2): track 0.00 -> 31.8 mm
- net Net-(R12-Pad2): track 0.00 -> 31.3 mm
- net Net-(F5-Pad2): track 24.9 -> 0.00 mm
- net Net-(F6-Pad2): track 23.9 -> 0.00 mm
- net Net-(F5-Pad1): track 2.67 -> 0.00 mm
- net Net-(F3-Pad1): track 2.10 -> 0.00 mm
- net Net-(F6-Pad1): track 2.03 -> 0.00 mm
- net Net-(F4-Pad1): track 2.03 -> 0.00 mm
- net 220VAC(L): track 69.4 -> 71.3 mm
Other:
- outline, holes or cut-outs redrawn
- board text added: "L"
- board text added: "N"
- board text removed: "5V"
- board text removed: "Ammeter Jumper"
- board text removed: "F-400mA"
- board text removed: "L 230V"
- board text removed: "L(VAC)"
- board text removed: "N 230V"
- board text removed: "N(VAC)"

Commit message: sent to JLPC
Parts:
- removed J8: 1017505, 1017505_updated_pretty:1017505_pretty
- added C12: 100nF, Capacitor_SMD:C_0805_2012Metric_Pad1.15x1.40mm_HandSolder, F.Cu at (188.7, 147.9)
- added C13: 22uF, Capacitor_Tantalum_SMD:CP_EIA-3528-21_Kemet-B_Pad1.50x2.35mm_HandSolder, F.Cu at (185.9, 147.0)
- added D1: LED, LED_SMD:LED_0805_2012Metric_Pad1.15x1.40mm_HandSolder, F.Cu at (183.1, 147.9)
- added G***: LOGO, icons:led_6000dpi, F.Cu at (181.2, 147.8)
- added H4: MountingHole_Pad, MountingHole:MountingHole_3.2mm_M3_ISO14580_Pad, F.Cu at (132.3, 85.4)
- added H5: MountingHole_Pad, MountingHole:MountingHole_3.2mm_M3_ISO14580_Pad, F.Cu at (198.6, 85.4)
- added H6: MountingHole_Pad, MountingHole:MountingHole_3.2mm_M3_ISO14580_Pad, F.Cu at (132.3, 74.7)
- added J4: 2604-1104, wago-2604-1104:big_pads_2604-1104, F.Cu at (194.4, 79.1)
- added R1: 100Ω, Resistor_SMD:R_0805_2012Metric_Pad1.15x1.40mm_HandSolder, F.Cu at (190.7, 147.9)
- C1, C2, C3, C4, C5, C6, C7: value 0.1uF -> 100nF
- F1: value F250V -> 250V1A
- F2: value 250v-40mA -> 250v50mA
- J1: value 1017505 -> 2604-1104; footprint 1017505_updated_pretty:1017505_pretty -> wago-2604-1104:big_pads_2604-1104
- J3: value 1017505 -> 2604-1102; footprint 1017505_updated_pretty:1017505_pretty -> wago-2604-1102:big_pads_2604-1102
- K1, K2, K3, K4: footprint PCN:TE_Connectivity-PCN-124D3MHZ,000-0-0-MFG -> PCN:bigpads_TE_Connectivity-PCN-124D
- R9: value 150Ω -> 100Ω
- moved G*** 25.0 mm to (185.4, 122.0)
- moved K3 6.29 mm to (166.9, 97.7)
- moved F1 6.12 mm to (146.7, 89.2)
- moved G*** 5.84 mm to (185.4, 111.8)
- moved J3 4.89 mm to (146.7, 79.1)
- moved J1 4.83 mm to (170.1, 79.1)
- moved K4 4.70 mm to (172.3, 97.7)
- moved F2 4.58 mm to (134.6, 92.3), turned to 0 degrees
- moved RV1 1.90 mm to (132.6, 99.0)
- moved K2 0.41 mm to (161.5, 97.7)
- moved K1 0.17 mm to (156.1, 97.7)
- renumbered 22uF3 to C10, 22uF4 to C11, 22uF1 to C8, 22uF2 to C9
Connections:
- net Net-(F1-Pad1) renamed L_IN
- F2 pad 1: Net-(F2-Pad1) -> N_IN
- J3 pad 3: (no net) -> N_IN
- J3 pad 4: (no net) -> N_IN
- K3 pad 11: REO4 -> REO3
- K3 pad A1: REI4 -> REI3
- K4 pad 11: REO3 -> REO4
- K4 pad A1: REI3 -> REI4
- R11 pad 1: Sens2 -> Sens1
- R13 pad 1: Sens1 -> Sens2
- RA05.SK.277 pad 1: 220VAC(N) -> N_IN
- RV1 pad 1: 220VAC(N) -> N_IN
Routing:
- net N_IN: track 0.00 -> 47.9 mm
- net Net-(F2-Pad1): track 14.5 -> 0.00 mm
- net GND(5V): track 162.8 -> 176.0 mm
- net Net-(C12-Pad1): track 0.00 -> 7.62 mm
- net Net-(C12-Pad2): track 0.00 -> 6.79 mm
- net 220VAC(N): track 100.2 -> 94.3 mm
- net Sens4: track 13.8 -> 18.5 mm
- net Sens3: track 13.8 -> 18.2 mm
- net Sens1: track 13.8 -> 18.1 mm
- net 220VAC(L): track 71.3 -> 67.2 mm
- net Sens2: track 14.2 -> 18.1 mm
- net REO1: track 13.6 -> 17.6 mm
- net REO2: track 13.7 -> 17.4 mm
- net REO4: track 14.2 -> 17.7 mm
- net REO3: track 14.1 -> 17.5 mm
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Other:
- board size 74.9 x 84.3 mm -> 76.7 x 84.3 mm
- board text added: "GND 5V"
- board text added: "V.20211112.05"
- board text removed: "250V-1A"
- board text removed: "GND"
- board text removed: "V.20211030.04"
