File: demo-11-esphome-module/schematics-v13-new-relays/main-project/hamodule.sch (KiCad schematic (older format))
At the start: 57 parts, among them J1 1017505, J10 GND 3.3V, J11 Current Jumper, J2 ESP Relays, J3 1017505, J5 Conn_01x02, J6 ESP Sensors, J8 1017505, J9 Current Jumper, K1 PCN-124D3MHZ,000, K2 PCN-124D3MHZ,000, K3 PCN-124D3MHZ,000, K4 PCN-124D3MHZ,000, U1 ULN2003A, U2 LD1117S33TR_SOT223, U3 HCPL3700, U4 HCPL3700, U5 HCPL3700, U6 HCPL3700

Commit message: cleaning tags
Parts:
- removed F3, F4, F5, F6: Fuse, Fuse:Fuse_1210_3225Metric_Pad1.42x2.65mm_HandSolder, symbol Device:Fuse
- K1, K2, K3, K4: value PCN-124D3MHZ,000 -> PCN-105D
- R10, R11, R12, R13, R14, R15, R16, R17: value 39kΩ1w -> 39kΩ3w
Connections:
- net at R14.2: now also U4.1 (1_AC)
- net at U3.1 (1_AC): now also R16.2
- net at R12.2: now also U5.1 (1_AC)
- net at R10.2: now also U6.1 (1_AC)
Changed lines of the file:
@@
-$EndComp
-$Comp
-L Device:Fuse F3
-U 1 1 61742087
-P 9950 2650
-F 0 "F3" V 9753 2650 50  0000 C CNN
-F 1 "Fuse" V 10050 2650 50  0000 C CNN
-F 2 "Fuse:Fuse_1210_3225Metric_Pad1.42x2.65mm_HandSolder" V 9880 2650 50  0001 C CNN
-F 3 "https://www.distrelec.ch/en/resettable-smd-fuse-60v-400ma-bel-fuse-0zcg0020af2c/p/30127324?q=fuse+smd&pos=4&origPos=112&origPageSize=50&track=true" H 9950 2650 50  0001 C CNN
-F 4 "C207063" H 9950 2650 50  0001 C CNN "JLCPCB"
-	1    9950 2650
-	0    1    1    0
-$EndComp
-$Comp
-L Device:Fuse F4
-U 1 1 6174141D
-P 9950 3850
-F 0 "F4" V 9753 3850 50  0000 C CNN
-F 1 "Fuse" V 10050 3850 50  0000 C CNN
-F 2 "Fuse:Fuse_1210_3225Metric_Pad1.42x2.65mm_HandSolder" V 9880 3850 50  0001 C CNN
-F 3 "https://www.distrelec.ch/en/resettable-smd-fuse-60v-400ma-bel-fuse-0zcg0020af2c/p/30127324?q=fuse+smd&pos=4&origPos=112&origPageSize=50&track=true" H 9950 3850 50  0001 C CNN
-F 4 "C207063" H 9950 3850 50  0001 C CNN "JLCPCB"
-	1    9950 3850
-	0    1    1    0
-$EndComp
-$Comp
-L Device:Fuse F6
-U 1 1 6173B2BF
-P 9950 5850
-F 0 "F6" V 9753 5850 50  0001 C CNN
-F 1 "Fuse" V 10050 5850 50  0000 C CNN
-F 2 "Fuse:Fuse_1210_3225Metric_Pad1.42x2.65mm_HandSolder" V 9880 5850 50  0001 C CNN
-F 3 "https://www.distrelec.ch/en/resettable-smd-fuse-60v-400ma-bel-fuse-0zcg0020af2c/p/30127324?q=fuse+smd&pos=4&origPos=112&origPageSize=50&track=true" H 9950 5850 50  0001 C CNN
-F 4 "C207063" H 9950 5850 50  0001 C CNN "JLCPCB"
-	1    9950 5850
-	0    1    1    0
-$EndComp
-$Comp
-L Device:Fuse F5
-U 1 1 6173596B
-P 9950 4850
-F 0 "F5" V 9753 4850 50  0000 C CNN
-F 1 "Fuse" V 10050 4850 50  0000 C CNN
-F 2 "Fuse:Fuse_1210_3225Metric_Pad1.42x2.65mm_HandSolder" V 9880 4850 50  0001 C CNN
-F 3 "https://www.distrelec.ch/en/resettable-smd-fuse-60v-400ma-bel-fuse-0zcg0020af2c/p/30127324?q=fuse+smd&pos=4&origPos=112&origPageSize=50&track=true" H 9950 4850 50  0001 C CNN
-F 4 "C207063" H 9950 4850 50  0001 C CNN "JLCPCB"
-	1    9950 4850
-	0    1    1    0
 $EndComp
 $Comp
@@
 P 10250 4850
 F 0 "R12" V 10043 4850 50  0001 C CNN
-F 1 "39kΩ1w" V 10350 4850 50  0000 C CNN
+F 1 "39kΩ3w" V 10350 4850 50  0000 C CNN
 F 2 "Resistor_SMD:R_2512_6332Metric_Pad1.52x3.35mm_HandSolder" V 10180 4850 50  0001 C CNN
 F 3 "https://www.distrelec.ch/en/super-high-power-smd-resistor-2512-82kohm-3w-rnd-components-rnd-155sp123wf8202t2e/p/30150189?q=*&pos=1&origPos=3001&origPageSize=50&digitalDataLayerTerm=resistor&track=true" H 10250 4850 50  0001 C CNN
@@
 P 10250 5850
 F 0 "R10" V 10043 5850 50  0001 C CNN
-F 1 "39kΩ1w" V 10350 5900 50  0000 C CNN
+F 1 "39kΩ3w" V 10350 5900 50  0000 C CNN
 F 2 "Resistor_SMD:R_2512_6332Metric_Pad1.52x3.35mm_HandSolder" V 10180 5850 50  0001 C CNN
 F 3 "https://www.distrelec.ch/en/super-high-power-smd-resistor-2512-82kohm-3w-rnd-components-rnd-155sp123wf8202t2e/p/30150189?q=*&pos=1&origPos=3001&origPageSize=50&digitalDataLayerTerm=resistor&track=true" H 10250 5850 50  0001 C CNN
@@
 P 10250 2650
 F 0 "R16" V 10043 2650 50  0001 C CNN
-F 1 "39kΩ1w" V 10350 2650 50  0000 C CNN
+F 1 "39kΩ3w" V 10350 2650 50  0000 C CNN
 F 2 "Resistor_SMD:R_2512_6332Metric_Pad1.52x3.35mm_HandSolder" V 10180 2650 50  0001 C CNN
 F 3 "https://www.distrelec.ch/en/super-high-power-smd-resistor-2512-82kohm-3w-rnd-components-rnd-155sp123wf8202t2e/p/30150189?q=*&pos=1&origPos=3001&origPageSize=50&digitalDataLayerTerm=resistor&track=true" H 10250 2650 50  0001 C CNN
@@
 P 10250 3850
 F 0 "R14" V 10043 3850 50  0001 C CNN
-F 1 "39kΩ1w" V 10350 3850 50  0000 C CNN
+F 1 "39kΩ3w" V 10350 3850 50  0000 C CNN
 F 2 "Resistor_SMD:R_2512_6332Metric_Pad1.52x3.35mm_HandSolder" V 10180 3850 50  0001 C CNN
 F 3 "https://www.distrelec.ch/en/super-high-power-smd-resistor-2512-82kohm-3w-rnd-components-rnd-155sp123wf8202t2e/p/30150189?q=*&pos=1&origPos=3001&origPageSize=50&digitalDataLayerTerm=resistor&track=true" H 10250 3850 50  0001 C CNN
@@
 P 10550 5850
 F 0 "R17" V 10343 5850 50  0001 C CNN
-F 1 "39kΩ1w" V 10650 5900 50  0000 C CNN
+F 1 "39kΩ3w" V 10650 5900 50  0000 C CNN
 F 2 "Resistor_SMD:R_2512_6332Metric_Pad1.52x3.35mm_HandSolder" V 10480 5850 50  0001 C CNN
 F 3 "https://www.distrelec.ch/en/super-high-power-smd-resistor-2512-82kohm-3w-rnd-components-rnd-155sp123wf8202t2e/p/30150189?q=*&pos=1&origPos=3001&origPageSize=50&digitalDataLayerTerm=resistor&track=true" H 10550 5850 50  0001 C CNN
@@
 P 10550 4850
 F 0 "R15" V 10343 4850 50  0001 C CNN
-F 1 "39kΩ1w" V 10650 4900 50  0000 C CNN
+F 1 "39kΩ3w" V 10650 4900 50  0000 C CNN
 F 2 "Resistor_SMD:R_2512_6332Metric_Pad1.52x3.35mm_HandSolder" V 10480 4850 50  0001 C CNN
 F 3 "https://www.distrelec.ch/en/super-high-power-smd-resistor-2512-82kohm-3w-rnd-components-rnd-155sp123wf8202t2e/p/30150189?q=*&pos=1&origPos=3001&origPageSize=50&digitalDataLayerTerm=resistor&track=true" H 10550 4850 50  0001 C CNN
@@
 P 10550 3850
 F 0 "R13" V 10343 3850 50  0001 C CNN
-F 1 "39kΩ1w" V 10650 3900 50  0000 C CNN
+F 1 "39kΩ3w" V 10650 3900 50  0000 C CNN
 F 2 "Resistor_SMD:R_2512_6332Metric_Pad1.52x3.35mm_HandSolder" V 10480 3850 50  0001 C CNN
 F 3 "https://www.distrelec.ch/en/super-high-power-smd-resistor-2512-82kohm-3w-rnd-components-rnd-155sp123wf8202t2e/p/30150189?q=*&pos=1&origPos=3001&origPageSize=50&digitalDataLayerTerm=resistor&track=true" H 10550 3850 50  0001 C CNN
@@
 P 10550 2650
 F 0 "R11" V 10343 2650 50  0001 C CNN
-F 1 "39kΩ1w" V 10650 2700 50  0000 C CNN
+F 1 "39kΩ3w" V 10650 2700 50  0000 C CNN
 F 2 "Resistor_SMD:R_2512_6332Metric_Pad1.52x3.35mm_HandSolder" V 10480 2650 50  0001 C CNN
 F 3 "https://www.distrelec.ch/en/super-high-power-smd-resistor-2512-82kohm-3w-rnd-components-rnd-155sp123wf8202t2e/p/30150189?q=*&pos=1&origPos=3001&origPageSize=50&digitalDataLayerTerm=resistor&track=true" H 10550 2650 50  0001 C CNN
@@
 Text GLabel 5500 1900 2    50   UnSpc ~ 0
 220VAC(N)
-Connection ~ 9800 2650
 $Comp
 L power:PWR_FLAG #FLG0101
@@
 P 1450 2100
 F 0 "K1" H 1850 2325 50  0000 C CNN
-F 1 "PCN-124D3MHZ,000" H 1850 2234 50  0000 C CNN
+F 1 "PCN-105D" H 1850 2234 50  0000 C CNN
 F 2 "PCN:TE_Connectivity-PCN-124D3MHZ,000-0-0-MFG" H 1450 2500 50  0001 L CNN
 F 3 "https://www.te.com/commerce/DocumentDelivery/DDEController?Action=showdoc&DocId=Data+Sheet%7FPCN_series_relay_data_sheet_E%7F1217%7Fpdf%7FEnglish%7FENG_DS_PCN_series_relay_data_sheet_E_1217.pdf%7F3-1461491-6" H 1450 2600 50  0001 L CNN
@@
 P 1450 3250
 F 0 "K2" H 1850 3475 50  0000 C CNN
-F 1 "PCN-124D3MHZ,000" H 1850 3384 50  0000 C CNN
+F 1 "PCN-105D" H 1850 3384 50  0000 C CNN
 F 2 "PCN:TE_Connectivity-PCN-124D3MHZ,000-0-0-MFG" H 1450 3650 50  0001 L CNN
 F 3 "https://www.te.com/commerce/DocumentDelivery/DDEController?Action=showdoc&DocId=Data+Sheet%7FPCN_series_relay_data_sheet_E%7F1217%7Fpdf%7FEnglish%7FENG_DS_PCN_series_relay_data_sheet_E_1217.pdf%7F3-1461491-6" H 1450 3750 50  0001 L CNN
@@
 P 1500 4550
 F 0 "K4" H 1900 4775 50  0000 C CNN
-F 1 "PCN-124D3MHZ,000" H 1900 4684 50  0000 C CNN
+F 1 "PCN-105D" H 1900 4684 50  0000 C CNN
 F 2 "PCN:TE_Connectivity-PCN-124D3MHZ,000-0-0-MFG" H 1500 4950 50  0001 L CNN
 F 3 "https://www.te.com/commerce/DocumentDelivery/DDEController?Action=showdoc&DocId=Data+Sheet%7FPCN_series_relay_data_sheet_E%7F1217%7Fpdf%7FEnglish%7FENG_DS_PCN_series_relay_data_sheet_E_1217.pdf%7F3-1461491-6" H 1500 5050 50  0001 L CNN
@@
 P 1450 5750
 F 0 "K3" H 1850 5975 50  0000 C CNN
-F 1 "PCN-124D3MHZ,000" H 1850 5884 50  0000 C CNN
+F 1 "PCN-105D" H 1850 5884 50  0000 C CNN
 F 2 "PCN:TE_Connectivity-PCN-124D3MHZ,000-0-0-MFG" H 1450 6150 50  0001 L CNN
 F 3 "https://www.te.com/commerce/DocumentDelivery/DDEController?Action=showdoc&DocId=Data+Sheet%7FPCN_series_relay_data_sheet_E%7F1217%7Fpdf%7FEnglish%7FENG_DS_PCN_series_relay_data_sheet_E_1217.pdf%7F3-1461491-6" H 1450 6250 50  0001 L CNN
@@
 Text GLabel 6450 2850 2    50   Input ~ 0
 GND(5V)
+Wire Wire Line
+	9800 2650 10100 2650
+Connection ~ 9800 2650
+Wire Wire Line
+	10100 3850 9800 3850
+Connection ~ 9800 3850
+Wire Wire Line
+	10100 4850 9800 4850
+Connection ~ 9800 4850
+Wire Wire Line
+	9800 5850 10100 5850
+Connection ~ 9800 5850
 $EndSCHEMATC

Commit message: sent to JLPC
Parts:
- removed J1, J3, J8: 1017505, 1017505_updated_pretty:1017505_pretty, symbol phoenix-1017505:1017505
- added C12: 100nF, Capacitor_SMD:C_0805_2012Metric_Pad1.15x1.40mm_HandSolder, symbol Device:CP
- added C13: 22uF, Capacitor_Tantalum_SMD:CP_EIA-3528-21_Kemet-B_Pad1.50x2.35mm_HandSolder, symbol Device:CP_Small
- added D1: LED, LED_SMD:LED_0805_2012Metric_Pad1.15x1.40mm_HandSolder, symbol Device:LED
- added H4, H5, H6: MountingHole_Pad, MountingHole:MountingHole_3.2mm_M3_ISO14580_Pad, symbol Mechanical:MountingHole_Pad
- added J1, J4: 2604-1104, wago-2604-1104:big_pads_2604-1104, symbol wago-2604-1104:2604-1104
- added J3: 2604-1102, wago-2604-1102:big_pads_2604-1102, symbol wago-2604-1102:2604-1102
- added R1: 100Ω, Resistor_SMD:R_0805_2012Metric_Pad1.15x1.40mm_HandSolder, symbol Device:R
- C1, C2, C3, C4, C5, C6, C7: value 0.1uF -> 100nF; JLCPCB C235777 -> C28233
- F1: value F250V -> 250V1A
- F2: value 250v-40mA -> 250v50mA
- K1, K2: footprint PCN:TE_Connectivity-PCN-124D3MHZ,000-0-0-MFG -> PCN:bigpads_TE_Connectivity-PCN-124D; symbol eec:PCN-124D3MHZ,000 -> pcn-105D3:PCN-124D3MHZ,000
- K3: renamed from K4; footprint PCN:TE_Connectivity-PCN-124D3MHZ,000-0-0-MFG -> PCN:bigpads_TE_Connectivity-PCN-124D; symbol eec:PCN-124D3MHZ,000 -> pcn-105D3:PCN-124D3MHZ,000
- K4: renamed from K3; footprint PCN:TE_Connectivity-PCN-124D3MHZ,000-0-0-MFG -> PCN:bigpads_TE_Connectivity-PCN-124D; symbol eec:PCN-124D3MHZ,000 -> pcn-105D3:PCN-124D3MHZ,000
- R10, R11, R12, R13, R14, R15, R16, R17: JLCPCB C25723 -> C144424
- R9: value 150Ω -> 100Ω; JLCPCB C17471 -> C17408
- renumbered 22uF3 to C10, 22uF4 to C11, 22uF1 to C8, 22uF2 to C9
Connections:
- net 220VAC(N): no longer RA05.SK.277.1 (VAC_IN(N)), RV1.1
- net REO1: now also J1.7, J1.8
- net REO2: now also J1.5, J1.6
- net REO3: now also J1.3, J1.4
- net REO4: now also J1.1, J1.2
- net Sens1: now also R11.1, J4.7, J4.8; no longer R13.1
- net Sens2: now also R13.1, J4.5, J4.6; no longer R11.1
- net Sens3: now also J4.3, J4.4
- net Sens4: now also J4.1, J4.2
- net L_IN: now reaches F1.1
- net L_IN: now also J3.1, J3.2
- net N_IN: now reaches F2.1
- net N_IN: now also RA05.SK.277.1 (VAC_IN(N)), RV1.1, J3.3, J3.4
- new net: C12.2, C13.1, D1.1 (K)
- new net: C12.1, C13.2, D1.2 (A), R1.1
Other:
- moved on the sheet: F2
