File: PCB/schematics-v18/kicad/hamodule.kicad_sch (KiCad schematic)
At the start: 97 parts, among them J1 Conn_01x02_Male, J10 DoNotCon, J11 2604-1104, J12 2604-1104, J13 EspSense, J2 2604-1102, J3 GND|5V, J4 GND|3.3V, J5 Jumper, J6 Conn_01x02_Male, J7 Current Jumper, J8 EspRelays, J9 USB_C_Receptacle_USB2.0, K1 PCN-105D, K2 PCN-105D, K3 PCN-105D, K4 PCN-105D, Q1 SS8050-SMD, Q2 SS8050, U1 LD1117AV33_TO220, U2 ESP32-WROOM-32E, U3 CP2102N-A01-GQFN28, U4 ULN2003A, U5 LDA210-PDIP, U6 LDA210-PDIP, U7 SHT4x

Commit message: [V18] fab files + images + readme + [V1]  schematics image in readme
Parts:
- SW1, SW2: value (none) -> Switch; footprint (none) -> Button_Switch_SMD:SW_SPST_SKQG_WithStem
Other:
- note added: "TODO: - Capacitors are too large for USB standard. Tested it with several hubs and it works - USB shield should probably not be connected to GND. It works with or without the connecting resistor"
- note removed: "TODO: - Do not add Capacitors to the LD1117, because USB inrush limitations - Should USB Shield be connected to GND?"
Changed lines of the file:
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@@
     (effects (font (size 1.27 1.27)) (justify left bottom))
   )
-  (text "TODO:\n- Do not add Capacitors to the LD1117, because USB inrush limitations\n- Should USB Shield be connected to GND?"
+  (text "TODO:\n- Capacitors are too large for USB standard. Tested it with several hubs and it works\n- USB shield should probably not be connected to GND. It works with or without the connecting resistor"
     (at 179.07 179.07 0)
     (effects (font (size 1.27 1.27)) (justify left bottom))
@@
     (in_bom yes) (on_board yes)
     (property "Reference" "SW1" (id 0) (at 223.52 115.57 0))
-    (property "Value" "" (id 1) (at 223.52 116.9924 0)
-      (effects (font (size 1.27 1.27)) hide)
-    )
-    (property "Footprint" "" (id 2) (at 223.52 116.84 0)
+    (property "Value" "Switch" (id 1) (at 223.52 116.9924 0)
+      (effects (font (size 1.27 1.27)) hide)
+    )
+    (property "Footprint" "Button_Switch_SMD:SW_SPST_SKQG_WithStem" (id 2) (at 223.52 116.84 0)
       (effects (font (size 1.27 1.27)) hide)
     )
@@
     (in_bom yes) (on_board yes)
     (property "Reference" "SW2" (id 0) (at 223.52 125.73 0))
-    (property "Value" "" (id 1) (at 223.52 127.1524 0)
-      (effects (font (size 1.27 1.27)) hide)
-    )
-    (property "Footprint" "" (id 2) (at 223.52 127 0)
-      (effects (font (size 1.27 1.27)) hide)
-    )
+    (property "Value" "Switch" (id 1) (at 223.52 127.1524 0)
+      (effects (font (size 1.27 1.27)) hide)
+    )
+    (property "Footprint" "Button_Switch_SMD:SW_SPST_SKQG_WithStem" (id 2) (at 223.52 127 0)
+      (effects (font (size 1.27 1.27)) hide)
+    )
