File: PCB/schematics-v19/kicad/hamodule.kicad_pcb (KiCad board)
At the start: 2 copper layers, 78.4 x 84.3 mm, 104 parts, among them J1 Conn_01x02_Male, J10 DoNotCon, J11 2604-1104, J12 2604-1104, J13 EspSense, J2 2604-1102, J3 GND|5V, J4 GND|3.3V, J5 Jumper, J6 Conn_01x02_Male, J7 Current Jumper, J8 EspRelays, J9 USB_C_Receptacle_USB2.0, K1 PCN-105D, K2 PCN-105D, K3 PCN-105D, K4 PCN-105D, Q1 SS8050-SMD, Q2 SS8050, SW1 Switch, SW2 Switch, U1 LD1117AV33_TO220, U2 ESP32-WROOM-32E, U3 CP2102N-A01-GQFN28, U4 ULN2003A, U5 LDA210-PDIP, U6 LDA210-PDIP, U7 SHT4x

Commit message: sent v19 to jlcpcb
Routing:
- net GND: track 284.5 -> 286.4 mm, vias 48 -> 49
Changed lines of the file:
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@@
       (drillshape 0)
       (scaleselection 1)
-      (outputdirectory "gerber/")
+      (outputdirectory "smt-assembly/")
     )
   )
@@
       ) (layer "B.SilkS") (width 0) (fill solid))
     (fp_poly (pts
-        (xy -6.356791 -0.421069)
-        (xy -6.370374 -0.434652)
-        (xy -6.383957 -0.421069)
-        (xy -6.370374 -0.407486)
-      ) (layer "B.SilkS") (width 0) (fill solid))
-    (fp_poly (pts
         (xy -10.730481 0.882888)
         (xy -10.744064 0.869305)
@@
       ) (layer "B.SilkS") (width 0) (fill solid))
     (fp_poly (pts
-        (xy -7.615472 -0.443707)
-        (xy -7.619201 -0.459857)
-        (xy -7.633583 -0.461818)
-        (xy -7.655943 -0.451878)
-        (xy -7.651693 -0.443707)
-        (xy -7.619454 -0.440456)
-      ) (layer "B.SilkS") (width 0) (fill solid))
-    (fp_poly (pts
-        (xy -9.508021 -0.421069)
-        (xy -9.521604 -0.434652)
-        (xy -9.535187 -0.421069)
-        (xy -9.521604 -0.407486)
-      ) (layer "B.SilkS") (width 0) (fill solid))
-    (fp_poly (pts
         (xy -9.779679 -0.855722)
         (xy -9.793262 -0.869304)
@@
       ) (layer "B.SilkS") (width 0) (fill solid))
     (fp_poly (pts
-        (xy -7.687914 -0.421069)
-        (xy -7.701497 -0.434652)
-        (xy -7.71508 -0.421069)
-        (xy -7.701497 -0.407486)
+        (xy -9.508021 -0.421069)
+        (xy -9.521604 -0.434652)
+        (xy -9.535187 -0.421069)
+        (xy -9.521604 -0.407486)
       ) (layer "B.SilkS") (width 0) (fill solid))
     (fp_poly (pts
@@
       ) (layer "B.SilkS") (width 0) (fill solid))
     (fp_poly (pts
+        (xy -7.076684 -0.258567)
+        (xy -6.91515 -0.318386)
+        (xy -6.786128 -0.356448)
+        (xy -6.674239 -0.376653)
+        (xy -6.5877 -0.382558)
+        (xy -6.499836 -0.385143)
+        (xy -6.462132 -0.388625)
+        (xy -6.470428 -0.395031)
+        (xy -6.520567 -0.406389)
+        (xy -6.533369 -0.409045)
+        (xy -6.692652 -0.429615)
+        (xy -6.83439 -0.417569)
+        (xy -6.914746 -0.396645)
+        (xy -6.98028 -0.373293)
+        (xy -7.041784 -0.347026)
+        (xy -7.089202 -0.323198)
+        (xy -7.11248 -0.307164)
+        (xy -7.101564 -0.304277)
+        (xy -7.076684 -0.310422)
+        (xy -7.022353 -0.326122)
+        (xy -7.076684 -0.281652)
+        (xy -7.131016 -0.237182)
+      ) (layer "B.SilkS") (width 0) (fill solid))
+    (fp_poly (pts
         (xy -8.837932 -1.421675)
         (xy -8.834681 -1.453915)
@@
       ) (layer "B.SilkS") (width 0) (fill solid))
     (fp_poly (pts
+        (xy -9.571408 -0.443707)
+        (xy -9.575137 -0.459857)
+        (xy -9.589518 -0.461818)
+        (xy -9.611879 -0.451878)
+        (xy -9.607629 -0.443707)
+        (xy -9.57539 -0.440456)
+      ) (layer "B.SilkS") (width 0) (fill solid))
+    (fp_poly (pts
         (xy -7.769411 -1.996684)
         (xy -7.782994 -2.010267)
@@
       ) (layer "B.SilkS") (width 0) (fill solid))
     (fp_poly (pts
+        (xy -7.615472 -0.443707)
+        (xy -7.619201 -0.459857)
+        (xy -7.633583 -0.461818)
+        (xy -7.655943 -0.451878)
+        (xy -7.651693 -0.443707)
+        (xy -7.619454 -0.440456)
+      ) (layer "B.SilkS") (width 0) (fill solid))
+    (fp_poly (pts
         (xy -8.828877 0.149412)
         (xy -8.84246 0.135829)
@@
       ) (layer "B.SilkS") (width 0) (fill solid))
     (fp_poly (pts
+        (xy -6.356791 -0.421069)
+        (xy -6.370374 -0.434652)
+        (xy -6.383957 -0.421069)
+        (xy -6.370374 -0.407486)
+      ) (layer "B.SilkS") (width 0) (fill solid))
+    (fp_poly (pts
         (xy -10.513155 -1.290374)
         (xy -10.526738 -1.303957)
@@
       ) (layer "B.SilkS") (width 0) (fill solid))
     (fp_poly (pts
-        (xy -7.076684 -0.258567)
-        (xy -6.91515 -0.318386)
-        (xy -6.786128 -0.356448)
-        (xy -6.674239 -0.376653)
-        (xy -6.5877 -0.382558)
-        (xy -6.499836 -0.385143)
-        (xy -6.462132 -0.388625)
-        (xy -6.470428 -0.395031)
-        (xy -6.520567 -0.406389)
-        (xy -6.533369 -0.409045)
-        (xy -6.692652 -0.429615)
-        (xy -6.83439 -0.417569)
-        (xy -6.914746 -0.396645)
-        (xy -6.98028 -0.373293)
-        (xy -7.041784 -0.347026)
-        (xy -7.089202 -0.323198)
-        (xy -7.11248 -0.307164)
-        (xy -7.101564 -0.304277)
-        (xy -7.076684 -0.310422)
-        (xy -7.022353 -0.326122)
-        (xy -7.076684 -0.281652)
-        (xy -7.131016 -0.237182)
-      ) (layer "B.SilkS") (width 0) (fill solid))
-    (fp_poly (pts
         (xy -9.033161 2.081165)
         (xy -8.9872 1.997684)
@@
       ) (layer "B.SilkS") (width 0) (fill solid))
     (fp_poly (pts
-        (xy -9.571408 -0.443707)
-        (xy -9.575137 -0.459857)
-        (xy -9.589518 -0.461818)
-        (xy -9.611879 -0.451878)
-        (xy -9.607629 -0.443707)
-        (xy -9.57539 -0.440456)
+        (xy -7.687914 -0.421069)
+        (xy -7.701497 -0.434652)
+        (xy -7.71508 -0.421069)
+        (xy -7.701497 -0.407486)
       ) (layer "B.SilkS") (width 0) (fill solid))
     (fp_poly (pts
@@
   (segment (start 193.8465 147.6435) (end 193.8465 147.8925) (width 1) (layer "F.Cu") (net 39))
   (segment (start 189.5983 136.7409) (end 189.5729 136.7663) (width 1) (layer "F.Cu") (net 39))
+  (segment (start 153.85 125.1) (end 153.85 123.85) (width 1) (layer "F.Cu") (net 39))
   (segment (start 182.1815 134.8613) (end 182.1815 138.6205) (width 1) (layer "F.Cu") (net 39))
   (segment (start 173.228 146.812) (end 173.228 148.045) (width 1) (layer "F.Cu") (net 39))
@@
   (segment (start 186.3979 132.2705) (end 186.3979 133.1849) (width 1) (layer "F.Cu") (net 39))
   (segment (start 157.612099 140.708899) (end 157.612099 140.871801) (width 0.6) (layer "F.Cu") (net 39))
+  (segment (start 153.85 123.85) (end 154.3 123.4) (width 1) (layer "F.Cu") (net 39))
   (segment (start 186.3725 136.4935) (end 186.3655 136.4865) (width 1) (layer "F.Cu") (net 39))
   (segment (start 195.886674 121.06272) (end 194.385074 122.56432) (width 1) (layer "F.Cu") (net 39))
@@
   (via (at 171.9 131.3) (size 0.8) (drill 0.4) (layers "F.Cu" "B.Cu") (net 39))
   (via (at 159.7965 137.9995) (size 0.8) (drill 0.4) (layers "F.Cu" "B.Cu") (net 39))
+  (via (at 154.3 123.4) (size 0.8) (drill 0.4) (layers "F.Cu" "B.Cu") (net 39))
   (via (at 160.9225 137.9741) (size 0.8) (drill 0.4) (layers "F.Cu" "B.Cu") (net 39))
   (via (at 160.9225 136.8565) (size 0.8) (drill 0.4) (layers "F.Cu" "B.Cu") (net 39))
