File: PCB/schematics-v22/kicad/hamodule.kicad_pcb (KiCad board)
At the start: 2 copper layers, 78.4 x 84.3 mm, 103 parts, among them J1 GND|5V, J10 Serial, J11 USB_C_Receptacle_USB2.0, J12 2604-1104, J13 EspSense, J2 2604-1102, J3 I2C, J4 13|12, J5 9|3|16, J6 GND|3.3V, J7 Current Jumper, J8 EspRelays, J9 2604-1104, K1 AQG12205, K2 AQG12205, K3 AQG12205, K4 AQG12205, SW1 Switch, SW2 Switch, SW3 USB | PS, U1 LD1117AV33, U2 ESP32-S3-WROOM-2, U3 ULN2003A, U4 USBLC6-2SC6, U5 LDA210-PDIP, U6 LDA210-PDIP, U7 SHT4x

Commit message: gerbers + fixing silkscreen
Changed lines of the file:
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@@
   (net 70 "Net-(J11-PadA7)")
   (net 71 "unconnected-(U2-Pad4)")
-  (net 72 "Net-(U4-Pad5)")
+  (net 72 "Net-(D3-Pad2)")
   (net 73 "Net-(J11-PadA5)")
   (net 74 "unconnected-(J11-PadA8)")
@@
     (property "Sheetname" "")
     (attr smd)
-    (fp_text reference "R11" (at 2.54 -0.3302) (layer "F.SilkS")
+    (fp_text reference "R11" (at 2.147 -0.0162 90) (layer "F.SilkS")
       (effects (font (size 0.6 0.6) (thickness 0.15)))
     )
@@
       (net 31 "VBUS") (pinfunction "K") (pintype "passive"))
     (pad "2" smd rect (at 1.05 0) (size 0.6 0.45) (layers "F.Cu" "F.Paste" "F.Mask")
-      (net 72 "Net-(U4-Pad5)") (pinfunction "A") (pintype "passive"))
+      (net 72 "Net-(D3-Pad2)") (pinfunction "A") (pintype "passive"))
     (model "${KICAD6_3DMODEL_DIR}/Diode_SMD.3dshapes/D_SOD-323.wrl"
       (offset (xyz 0 0 0))
@@
       (net 32 "GND") (pinfunction "GND") (pintype "passive"))
     (pad "A4" smd rect (at -2.45 -4.045) (size 0.6 1.45) (layers "F.Cu" "F.Paste" "F.Mask")
-      (net 72 "Net-(U4-Pad5)") (pinfunction "VBUS") (pintype "passive"))
+      (net 72 "Net-(D3-Pad2)") (pinfunction "VBUS") (pintype "passive"))
     (pad "A5" smd rect (at -1.25 -4.045) (size 0.3 1.45) (layers "F.Cu" "F.Paste" "F.Mask")
       (net 73 "Net-(J11-PadA5)") (pinfunction "CC1") (pintype "bidirectional"))
@@
       (net 74 "unconnected-(J11-PadA8)") (pinfunction "SBU1") (pintype "bidirectional+no_connect"))
     (pad "A9" smd rect (at 2.45 -4.045) (size 0.6 1.45) (layers "F.Cu" "F.Paste" "F.Mask")
-      (net 72 "Net-(U4-Pad5)") (pinfunction "VBUS") (pintype "passive"))
+      (net 72 "Net-(D3-Pad2)") (pinfunction "VBUS") (pintype "passive"))
     (pad "A12" smd rect (at 3.25 -4.045) (size 0.6 1.45) (layers "F.Cu" "F.Paste" "F.Mask")
       (net 32 "GND") (pinfunction "GND") (pintype "passive"))
@@
       (net 32 "GND") (pinfunction "GND") (pintype "passive"))
     (pad "B4" smd rect (at 2.45 -4.045) (size 0.6 1.45) (layers "F.Cu" "F.Paste" "F.Mask")
-      (net 72 "Net-(U4-Pad5)") (pinfunction "VBUS") (pintype "passive"))
+      (net 72 "Net-(D3-Pad2)") (pinfunction "VBUS") (pintype "passive"))
     (pad "B5" smd rect (at 1.75 -4.045) (size 0.3 1.45) (layers "F.Cu" "F.Paste" "F.Mask")
       (net 75 "Net-(J11-PadB5)") (pinfunction "CC2") (pintype "bidirectional"))
@@
       (net 80 "unconnected-(J11-PadB8)") (pinfunction "SBU2") (pintype "bidirectional+no_connect"))
     (pad "B9" smd rect (at -2.45 -4.045) (size 0.6 1.45) (layers "F.Cu" "F.Paste" "F.Mask")
-      (net 72 "Net-(U4-Pad5)") (pinfunction "VBUS") (pintype "passive"))
+      (net 72 "Net-(D3-Pad2)") (pinfunction "VBUS") (pintype "passive"))
     (pad "B12" smd rect (at -3.25 -4.045) (size 0.6 1.45) (layers "F.Cu" "F.Paste" "F.Mask")
       (net 32 "GND") (pinfunction "GND") (pintype "passive"))
@@
     (property "Sheetname" "")
     (attr smd)
-    (fp_text reference "C16" (at -2.5035 0.4572) (layer "F.SilkS")
+    (fp_text reference "C16" (at -2.1045 0.1382 90) (layer "F.SilkS")
       (effects (font (size 0.6 0.6) (thickness 0.15)))
     )
@@
       (net 26 "D+") (pinfunction "I/O2") (pintype "passive"))
     (pad "5" smd roundrect (at 1.1375 0 90) (size 1.325 0.6) (layers "F.Cu" "F.Paste" "F.Mask") (roundrect_rratio 0.25)
-      (net 72 "Net-(U4-Pad5)") (pinfunction "VBUS") (pintype "passive"))
+      (net 72 "Net-(D3-Pad2)") (pinfunction "VBUS") (pintype "passive"))
     (pad "6" smd roundrect (at 1.1375 -0.95 90) (size 1.325 0.6) (layers "F.Cu" "F.Paste" "F.Mask") (roundrect_rratio 0.25)
       (net 27 "D-") (pinfunction "I/O1") (pintype "passive"))
@@
     (property "Sheetname" "")
     (attr smd)
-    (fp_text reference "R12" (at -2.5024 0.508) (layer "F.SilkS")
+    (fp_text reference "R12" (at -2.1234 0.013 90) (layer "F.SilkS")
       (effects (font (size 0.6 0.6) (thickness 0.15)))
     )
@@
     (property "Sheetname" "")
     (attr smd)
-    (fp_text reference "C15" (at 2.5411 -0.2032 180) (layer "F.SilkS")
+    (fp_text reference "C15" (at 2.1981 0.2098 270) (layer "F.SilkS")
       (effects (font (size 0.6 0.6) (thickness 0.15)))
     )
@@
     (property "Sheetname" "")
     (attr smd)
-    (fp_text reference "C20" (at 0 -1.68) (layer "F.SilkS")
-      (effects (font (size 1 1) (thickness 0.15)))
+    (fp_text reference "C20" (at -2.3325 -0.06 90) (layer "F.SilkS")
+      (effects (font (size 0.6 0.6) (thickness 0.15)))
     )
-    (fp_text value "NC" (at 0 1.68) (layer "F.Fab")
-      (effects (font (size 1 1) (thickness 0.15)))
+    (fp_text value "NC" (at 0 1.68) (layer "F.SilkS") hide
+      (effects (font (size 0.6 0.6) (thickness 0.15)))
     )
     (fp_text user "${REFERENCE}" (at 0 0) (layer "F.Fab")
@@
     (fp_line (start -1 -0.625) (end 1 -0.625) (layer "F.Fab") (width 0.1))
     (fp_line (start 1 0.625) (end -1 0.625) (layer "F.Fab") (width 0.1))
-    (pad "1" smd roundrect (at -1.0375 0) (size 1.175 1.45) (layers "F.Cu" "F.Paste" "F.Mask") (roundrect_rratio 0.212766)
+    (pad "1" smd roundrect (at -1.0375 0) (size 1.175 1.45) (layers "F.Cu" "F.Paste" "F.Mask") (roundrect_rratio 0.2127659574)
       (net 3 "3.3V+") (pintype "passive"))
-    (pad "2" smd roundrect (at 1.0375 0) (size 1.175 1.45) (layers "F.Cu" "F.Paste" "F.Mask") (roundrect_rratio 0.212766)
+    (pad "2" smd roundrect (at 1.0375 0) (size 1.175 1.45) (layers "F.Cu" "F.Paste" "F.Mask") (roundrect_rratio 0.2127659574)
       (net 32 "GND") (pintype "passive"))
     (model "${KICAD6_3DMODEL_DIR}/Capacitor_SMD.3dshapes/C_0805_2012Metric.wrl"
@@
     (fp_line (start 1.6 -0.8) (end -1.6 -0.8) (layer "B.Fab") (width 0.1))
     (fp_line (start 1.6 0.8) (end 1.6 -0.8) (layer "B.Fab") (width 0.1))
-    (pad "1" smd roundrect (at -1.5625 0) (size 1.325 1.8) (layers "B.Cu" "B.Paste" "B.Mask") (roundrect_rratio 0.188679)
+    (pad "1" smd roundrect (at -1.5625 0) (size 1.325 1.8) (layers "B.Cu" "B.Paste" "B.Mask") (roundrect_rratio 0.1886792453)
       (net 3 "3.3V+") (pintype "passive"))
-    (pad "2" smd roundrect (at 1.5625 0) (size 1.325 1.8) (layers "B.Cu" "B.Paste" "B.Mask") (roundrect_rratio 0.188679)
+    (pad "2" smd roundrect (at 1.5625 0) (size 1.325 1.8) (layers "B.Cu" "B.Paste" "B.Mask") (roundrect_rratio 0.1886792453)
       (net 32 "GND") (pintype "passive"))
     (model "${KICAD6_3DMODEL_DIR}/Capacitor_SMD.3dshapes/C_1206_3216Metric.wrl"
