File: PCB/schematics-v22-jlcpcb/kicad/hamodule.kicad_pcb (KiCad board)
At the start: 2 copper layers, 78.4 x 84.3 mm, 103 parts, among them J1 GND|5V, J10 Serial, J11 USB_C_Receptacle_USB2.0, J12 2604-1104, J13 EspSense, J2 2604-1102, J3 I2C, J4 13|12, J5 9|3|16, J6 GND|3.3V, J7 Current Jumper, J8 EspRelays, J9 2604-1104, K1 AQG12205, K2 AQG12205, K3 AQG12205, K4 AQG12205, SW1 Switch, SW2 Switch, SW3 USB | PS, U1 LD1117AV33, U2 ESP32-S3-WROOM-2, U3 ULN2003A, U4 USBLC6-2SC6, U5 LDA210-PDIP, U6 LDA210-PDIP, U7 SHT4x

Commit message: testing changes
Parts:
- removed F2, F9: Fuse, RST-80-AMMO:FUSE_RST-1-BULK
- removed K1: AQG12205, AQG12205:AQG12205
- added D8: LED, LED_SMD:LED_0805_2012Metric_Pad1.15x1.40mm_HandSolder, F.Cu at (60.8, 72.9)
- added R27: 100Ω, Resistor_SMD:R_0805_2012Metric_Pad1.20x1.40mm_HandSolder, F.Cu at (60.8, 75.1)
- added R28: 150kΩ1w, Resistor_SMD:R_2512_6332Metric_Pad1.40x3.35mm_HandSolder, F.Cu at (98.9, 50.5)
Connections:
- J9 pad 7: Net-(F2-Pad2) -> unconnected-(J9-Pad7)
- J9 pad 8: Net-(F2-Pad2) -> unconnected-(J9-Pad8)
- U3 pad 13: Net-(K1-Pad1) -> unconnected-(U3-Pad13)
Routing:
- net Net-(K1-Pad1): track 16.3 -> 0.00 mm
- net unconnected-(J9-Pad7): track 0.00 -> 13.3 mm
- net Net-(F2-Pad2): track 13.3 -> 0.00 mm
- net Net-(F2-Pad1): track 5.09 -> 0.00 mm
- net (no net): track 0.00 -> 5.09 mm
- net Net-(D8-Pad2): track 0.00 -> 2.99 mm
- net GND: track 189.1 -> 191.5 mm, vias 45 -> 46
- net 5V+: track 74.3 -> 73.2 mm

Commit message: more changes
Parts:
- added D8: LED, LED_SMD:LED_0805_2012Metric_Pad1.15x1.40mm_HandSolder, F.Cu at (60.8, 79.1)
- added R27: 100Ω, Resistor_SMD:R_0805_2012Metric_Pad1.20x1.40mm_HandSolder, F.Cu at (60.8, 77.1)
Routing:
- net (no net): track 5.09 -> 9.15 mm, vias 0 -> 1
Changed lines of the file:
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@@
     )
   )
+  (footprint "LED_SMD:LED_0805_2012Metric_Pad1.15x1.40mm_HandSolder" (layer "F.Cu")
+    (at 60.833 79.121)
+    (descr "LED SMD 0805 (2012 Metric), square (rectangular) end terminal, IPC_7351 nominal, (Body size source: https://docs.google.com/spreadsheets/d/1BsfQQcO9C6DZCsRaXUlFlo91Tg2WpOkGARC1WS5S8t0/edit?usp=sharing), generated with kicad-footprint-generator")
+    (tags "LED handsolder")
+    (property "JLCPCB" "C2297")
+    (property "LCSC" "C2297")
+    (property "Sheetfile" "hamodule.kicad_sch")
+    (property "Sheetname" "")
+    (attr smd)
+    (fp_text reference "D8" (at 0 -1.65) (layer "F.SilkS")
+      (effects (font (size 1 1) (thickness 0.15)))
+    )
+    (fp_text value "LED" (at 0 1.65) (layer "F.Fab")
+      (effects (font (size 1 1) (thickness 0.15)))
+    )
+    (fp_text user "${REFERENCE}" (at 0 0) (layer "F.Fab")
+      (effects (font (size 0.5 0.5) (thickness 0.08)))
+    )
+    (fp_line (start -1.86 -0.96) (end -1.86 0.96) (layer "F.SilkS") (width 0.12))
+    (fp_line (start -1.86 0.96) (end 1 0.96) (layer "F.SilkS") (width 0.12))
+    (fp_line (start 1 -0.96) (end -1.86 -0.96) (layer "F.SilkS") (width 0.12))
+    (fp_line (start 1.85 -0.95) (end 1.85 0.95) (layer "F.CrtYd") (width 0.05))
+    (fp_line (start 1.85 0.95) (end -1.85 0.95) (layer "F.CrtYd") (width 0.05))
+    (fp_line (start -1.85 0.95) (end -1.85 -0.95) (layer "F.CrtYd") (width 0.05))
+    (fp_line (start -1.85 -0.95) (end 1.85 -0.95) (layer "F.CrtYd") (width 0.05))
+    (fp_line (start -1 0.6) (end 1 0.6) (layer "F.Fab") (width 0.1))
+    (fp_line (start -0.7 -0.6) (end -1 -0.3) (layer "F.Fab") (width 0.1))
+    (fp_line (start -1 -0.3) (end -1 0.6) (layer "F.Fab") (width 0.1))
+    (fp_line (start 1 -0.6) (end -0.7 -0.6) (layer "F.Fab") (width 0.1))
+    (fp_line (start 1 0.6) (end 1 -0.6) (layer "F.Fab") (width 0.1))
+    (pad "1" smd roundrect (at -1.025 0) (size 1.15 1.4) (layers "F.Cu" "F.Paste" "F.Mask") (roundrect_rratio 0.217391)
+      (pinfunction "K") (pintype "passive"))
+    (pad "2" smd roundrect (at 1.025 0) (size 1.15 1.4) (layers "F.Cu" "F.Paste" "F.Mask") (roundrect_rratio 0.217391)
+      (pinfunction "A") (pintype "passive"))
+    (model "${KICAD6_3DMODEL_DIR}/LED_SMD.3dshapes/LED_0805_2012Metric.wrl"
+      (offset (xyz 0 0 0))
+      (scale (xyz 1 1 1))
+      (rotate (xyz 0 0 0))
+    )
+  )
   (footprint "Resistor_SMD:R_0603_1608Metric_Pad0.98x0.95mm_HandSolder" (layer "F.Cu")
     (at 95.9001 83.8962)
@@
     )
   )
+  (footprint "Resistor_SMD:R_0805_2012Metric_Pad1.20x1.40mm_HandSolder" (layer "F.Cu")
+    (at 60.833 77.089)
+    (descr "Resistor SMD 0805 (2012 Metric), square (rectangular) end terminal, IPC_7351 nominal with elongated pad for handsoldering. (Body size source: IPC-SM-782 page 72, https://www.pcb-3d.com/wordpress/wp-content/uploads/ipc-sm-782a_amendment_1_and_2.pdf), generated with kicad-footprint-generator")
+    (tags "resistor handsolder")
+    (property "JLCPCB" "C17408")
+    (property "LCSC" "C17408")
+    (property "Sheetfile" "hamodule.kicad_sch")
+    (property "Sheetname" "")
+    (attr smd)
+    (fp_text reference "R27" (at 0 -1.65) (layer "F.SilkS")
+      (effects (font (size 1 1) (thickness 0.15)))
+    )
+    (fp_text value "100Ω" (at 0 1.65) (layer "F.Fab")
+      (effects (font (size 1 1) (thickness 0.15)))
+    )
+    (fp_text user "${REFERENCE}" (at 0 0) (layer "F.Fab")
+      (effects (font (size 0.5 0.5) (thickness 0.08)))
+    )
+    (fp_line (start -0.227064 -0.735) (end 0.227064 -0.735) (layer "F.SilkS") (width 0.12))
+    (fp_line (start -0.227064 0.735) (end 0.227064 0.735) (layer "F.SilkS") (width 0.12))
+    (fp_line (start 1.85 0.95) (end -1.85 0.95) (layer "F.CrtYd") (width 0.05))
+    (fp_line (start -1.85 -0.95) (end 1.85 -0.95) (layer "F.CrtYd") (width 0.05))
+    (fp_line (start 1.85 -0.95) (end 1.85 0.95) (layer "F.CrtYd") (width 0.05))
+    (fp_line (start -1.85 0.95) (end -1.85 -0.95) (layer "F.CrtYd") (width 0.05))
+    (fp_line (start 1 0.625) (end -1 0.625) (layer "F.Fab") (width 0.1))
+    (fp_line (start -1 -0.625) (end 1 -0.625) (layer "F.Fab") (width 0.1))
+    (fp_line (start 1 -0.625) (end 1 0.625) (layer "F.Fab") (width 0.1))
+    (fp_line (start -1 0.625) (end -1 -0.625) (layer "F.Fab") (width 0.1))
+    (pad "1" smd roundrect (at -1 0) (size 1.2 1.4) (layers "F.Cu" "F.Paste" "F.Mask") (roundrect_rratio 0.208333)
+      (pintype "passive"))
+    (pad "2" smd roundrect (at 1 0) (size 1.2 1.4) (layers "F.Cu" "F.Paste" "F.Mask") (roundrect_rratio 0.208333)
+      (pintype "passive"))
+    (model "${KICAD6_3DMODEL_DIR}/Resistor_SMD.3dshapes/R_0805_2012Metric.wrl"
+      (offset (xyz 0 0 0))
+      (scale (xyz 1 1 1))
+      (rotate (xyz 0 0 0))
+    )
+  )
   (footprint "Resistor_SMD:R_0603_1608Metric_Pad0.98x0.95mm_HandSolder" (layer "F.Cu")
     (at 69.68 103.69 90)
@@
   )
   (segment (start 59.817 52.959) (end 59.817 54.991) (width 2) (layer "F.Cu") (net 0))
+  (segment (start 61.833 79.096) (end 61.858 79.121) (width 0.2) (layer "F.Cu") (net 0))
   (segment (start 59.817 54.991) (end 61.976 57.15) (width 2) (layer "F.Cu") (net 0))
+  (segment (start 61.833 77.089) (end 61.833 79.096) (width 0.2) (layer "F.Cu") (net 0))
+  (segment (start 58.665 80.264) (end 58.2555 80.264) (width 0.2) (layer "F.Cu") (net 0))
+  (segment (start 59.808 79.121) (end 58.665 80.264) (width 0.2) (layer "F.Cu") (net 0))
+  (via (at 58.2555 80.264) (size 0.8) (drill 0.4) (layers "F.Cu" "B.Cu") (net 0))
   (segment (start 34.8391 88.805) (end 34.8391 79.5757) (width 3) (layer "F.Cu") (net 1))
   (segment (start 49.2038 65.211) (end 49.2038 63.3638) (width 3) (layer "F.Cu") (net 1))
