File: PCB/schematics-v22-jlcpcb/kicad/hamodule.kicad_sch (KiCad schematic)
At the start: 96 parts, among them J1 GND|5V, J10 Serial, J11 USB_C_Receptacle_USB2.0, J12 2604-1104, J13 EspSense, J2 2604-1102, J3 I2C, J4 13|12, J5 9|3|16, J6 GND|3.3V, J7 Current Jumper, J8 EspRelays, J9 2604-1104, K1 AQG12205, K2 AQG12205, K3 AQG12205, K4 AQG12205, SW1 Switch, SW2 Switch, SW3 USB | PS, U1 LD1117AV33, U2 ESP32-S3-WROOM-2, U3 ULN2003A, U4 USBLC6-2SC6, U5 LDA210-PDIP, U6 LDA210-PDIP, U7 SHT4x

Commit message: [v22] Migrating to k7; [v23] new one
Parts:
- J10, J3, J4: symbol Connector:Conn_01x02_Male -> Connector:Conn_01x02_Pin
- J11: footprint Connector_USB:USB_C_Receptacle_HRO_TYPE-C-31-M-12 -> Connector_USB:USB_C_Receptacle_G-Switch_GT-USB-7010ASV
- J13, J8: symbol Connector:Conn_01x04_Male -> Connector:Conn_01x04_Pin
- J5: symbol Connector:Conn_01x03_Male -> Connector:Conn_01x03_Pin
- J7: symbol Connector:Conn_01x02_Male -> Jumper:Jumper_2_Bridged
- SW1, SW2: footprint Button_Switch_SMD:SW_SPST_SKQG_WithStem -> Button_Switch_SMD:SW_SPST_TL3342
- SW3: symbol Switch:SW_DPDT_x2 -> Switch:SW_SPDT
Connections:
- net 3.3V+: now also J7.2 (B); no longer J7.1 (Pin_1)
- net at C10.1, C11.1, C8.1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: now also J7.1 (A); no longer J7.2 (Pin_2)
Other:
- moved on the sheet: C10, C11, C4, C6, C7, C8, C9, J1, J6
