File: PCB/schematics-v23/kicad/hamodule.kicad_sch (KiCad schematic)
At the start: 135 parts, among them J1 GND|5V, J10 Serial, J11 USB_C_Receptacle_USB2.0, J12 2604-1104, J14 2604-1104, J15 2604-1104, J2 2604-1102, J3 I2C, J4 13|12, J5 9|3|16, J6 GND|3.3V, J7 Current Jumper, J9 2604-1104, K1 AQG12205, K2 AQG12205, K3 AQG12205, K4 AQG12205, K5 AQG12205, K6 AQG12205, K7 AQG12205, K8 AQG12205, SW1 Switch, SW2 Switch, SW3 USB | PS, U1 LD1117AV33, U10 ULN2803A, U2 ESP32-S3-WROOM-2, U3 LDA210-PDIP, U4 USBLC6-2SC6, U5 LDA210-PDIP, U6 LDA210-PDIP, U7 SHT4x, U8 LDA210-PDIP, U9 MCP23017_SO

Commit message: [V23] In progress: 8 channels solution
Connections:
- net I1: now reaches F9.2, J12.1, J12.2
- net I2: now reaches F8.2, J12.3, J12.4
- net I3: now reaches F7.2, J12.5, J12.6
- net I4: now reaches F6.2, J12.7, J12.8
- net EspRel1: no longer names the net of U2.16 (GPIO46)
- net EspRel2: no longer names the net of U2.12 (GPIO8/TOUCH8/ADC1_CH7/SUBSPICS1)
- net EspRel3: no longer names the net of U2.11 (GPIO18/U1RXD/ADC2_CH7/CLK_OUT3)
- net EspRel4: no longer names the net of U2.10 (GPIO17/U1TXD/ADC2_CH6)
- net EspSens1: no longer names the net of U2.8 (GPIO15/U0RTS/ADC2_CH4/XTAL_32K_P)
- net EspSens2: no longer names the net of U2.7 (GPIO7/TOUCH7/ADC1_CH6)
- net EspSens3: no longer names the net of U2.6 (GPIO6/TOUCH6/ADC1_CH5)
- net EspSens4: no longer names the net of U2.5 (GPIO5/TOUCH5/ADC1_CH4)
- no-connect marks 17 -> 28
Other:
- moved on the sheet: C1, C10, C11, C12, C13, C15, C16, C17, C18, C19, C2, C20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

Commit message: [V23] Fixing MCP, Fixing most DRC & ERC errors. Updating to Kicad7 (netclases, footprints changes only in library)
Parts:
- added C25: 100nF, Capacitor_SMD:C_0603_1608Metric_Pad1.08x0.95mm_HandSolder, symbol Device:C_Polarized_Small
- added R43: 22Ω, Resistor_SMD:R_0603_1608Metric, symbol Device:R_Small
- J10: value Serial -> Tx|Rx; symbol Connector:Conn_01x02_Male -> Connector:Conn_01x02_Pin; Field4 Rx | Tx -> (none)
- J11: footprint Connector_USB:USB_C_Receptacle_HRO_TYPE-C-31-M-12 -> usb-c:USB_C_Receptacle_HRO_TYPE-C-31-M-12
- J3: value I2C -> Sda|Scl; symbol Connector:Conn_01x02_Male -> Connector:Conn_01x02_Pin; Field4 SDA|SCL -> (none)
- J4: symbol Connector:Conn_01x02_Male -> Connector:Conn_01x02_Pin; Field4 12|13 -> (none)
- J5: symbol Connector:Conn_01x03_Male -> Connector:Conn_01x03_Pin
- J7: value Current Jumper -> Conn_01x02_Pin; symbol Connector:Conn_01x02_Male -> Connector:Conn_01x02_Pin
- SW1: footprint Button_Switch_SMD:SW_SPST_SKQG_WithStem -> hamodule_SW_SPST_SKQG_WithStem:SW_SPST_SKQG_WithStem; PcbText (none) -> Reset
- SW2: footprint Button_Switch_SMD:SW_SPST_SKQG_WithStem -> hamodule_SW_SPST_SKQG_WithStem:SW_SPST_SKQG_WithStem; PcbText (none) -> Boot
- SW3: symbol Switch:SW_DPDT_x2 -> Switch:SW_SPDT; PcbText USB|PS -> (none)
Connections:
- net 3.3V+: now also C25.1, R43.1
- net GND: now also C25.2
- net at U9.18 (~{RESET}): now also R43.2
- net I1: no longer names the net of F9.2, J12.1, J12.2
- net I2: no longer names the net of F8.2, J12.3, J12.4
- net I3: no longer names the net of F7.2, J12.5, J12.6
- net I4: no longer names the net of F6.2, J12.7, J12.8
- no-connect marks 28 -> 27
Other:
- moved on the sheet: C15, C16, C17, C18, C4, C6, C7, F10, F11, F12, F13, F6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
