File: PCB/schematics-v25-2/kicad/hamodule.kicad_sch (KiCad schematic)
At the start: 190 parts, among them J1 GND|5V, J10 Tx|Rx, J11 Sda|Scl, J12 3|9, J13 13|12, J14 3.3v|GND|7|15, J15 2604-1104, J16 2604-1104, J17 TestPoint, J19 TestPoint, J2 2604-1102, J3 USB_C_Receptacle_USB2.0, J4 GND|3.3V, J5 Conn_01x02_Pin, J6 2604-1104, J7 2604-1104, J8 5v|GND|Do, J9 Screen, K1 AQG22205, K2 AQG22205, K3 AQG22205, K4 AQG22205, K5 AQG22205, K6 AQG22205, K7 AQG22205, K8 AQG22205, SW1 USB | PS, SW2 Reset, SW3 Boot, U1 LD1117AV33, U10 SN74LV1T34DBV, U11 ULN2803A, U12 TCAL6416, U14 74AHC1G04, U2 USBLC6-2SC6, U3 ESP32-S3-WROOM-2, U4 LDA210, U5 LDA210, U6 LDA210, U7 LDA210, U8 SHT4x, U9 SN74LVCH8T245

Commit message: minor changes
Parts:
- added R59: 10kΩ, Resistor_SMD:R_0603_1608Metric_Pad0.98x0.95mm_HandSolder, symbol Device:R
- JP2, JP3: footprint Jumper:SolderJumper-2_P1.3mm_Bridged2Bar_RoundedPad1.0x1.5mm -> Jumper:SolderJumper-2_P1.3mm_Open_RoundedPad1.0x1.5mm; symbol Jumper:SolderJumper_2_Bridged -> Jumper:SolderJumper_2_Open
Connections:
- net GND: now also R59.1
- net OUT_ENABLE: now also R59.2
Other:
- moved on the sheet: R61
Changed lines of the file:
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@@
 	)
 	(rectangle
+		(start 248.92 69.85)
+		(end 261.62 82.55)
+		(stroke
+			(width 0)
+			(type dash)
+			(color 255 0 255 1)
+		)
+		(fill
+			(type none)
+		)
+	)
+	(rectangle
 		(start 12.7 104.14)
 		(end 134.62 184.15)
@@
 		)
 	)
+	(text "Not required"
+		(exclude_from_sim no)
+		(at 255.524 81.026 0)
+		(effects
+			(font
+				(size 1.27 1.27)
+				(color 255 0 255 1)
+			)
+		)
+	)
 	(text "Temperature Sensor"
 		(exclude_from_sim no)
@@
 	)
 	(junction
+		(at 29.21 228.6)
+		(diameter 0)
+		(color 0 0 0 0)
+	)
+	(junction
 		(at 278.13 128.27)
 		(diameter 0)
@@
 	(wire
 		(pts
+			(xy 29.21 228.6) (xy 31.75 228.6)
+		)
+		(stroke
+			(width 0)
+			(type default)
+		)
+	)
+	(wire
+		(pts
 			(xy 53.34 88.9) (xy 53.34 92.71)
 		)
@@
 	(wire
 		(pts
-			(xy 261.62 73.66) (xy 265.43 73.66)
+			(xy 260.35 73.66) (xy 265.43 73.66)
 		)
 		(stroke
@@
 	(wire
 		(pts
+			(xy 27.94 228.6) (xy 29.21 228.6)
+		)
+		(stroke
+			(width 0)
+			(type default)
+		)
+	)
+	(wire
+		(pts
 			(xy 180.34 156.21) (xy 184.15 156.21)
 		)
@@
 	(wire
 		(pts
-			(xy 262.89 83.82) (xy 265.43 83.82)
+			(xy 262.89 85.09) (xy 265.43 85.09)
 		)
 		(stroke
@@
 	(wire
 		(pts
+			(xy 31.75 228.6) (xy 31.75 246.38)
+		)
+		(stroke
+			(width 0)
+			(type default)
+		)
+	)
+	(wire
+		(pts
 			(xy 304.8 128.27) (xy 307.34 128.27)
 		)
@@
 	(wire
 		(pts
-			(xy 265.43 83.82) (xy 265.43 82.55)
+			(xy 265.43 85.09) (xy 265.43 82.55)
 		)
 		(stroke
@@
 	(wire
 		(pts
-			(xy 261.62 78.74) (xy 261.62 73.66)
+			(xy 260.35 78.74) (xy 260.35 73.66)
 		)
 		(stroke
@@
 	(wire
 		(pts
-			(xy 251.46 78.74) (xy 254 78.74)
+			(xy 251.46 78.74) (xy 252.73 78.74)
 		)
 		(stroke
@@
 	(wire
 		(pts
+			(xy 31.75 246.38) (xy 44.45 246.38)
+		)
+		(stroke
+			(width 0)
+			(type default)
+		)
+	)
+	(wire
+		(pts
 			(xy 261.62 228.6) (xy 276.86 228.6)
 		)
@@
 	(global_label "OUT_ENABLE"
 		(shape input)
-		(at 262.89 83.82 180)
+		(at 262.89 85.09 180)
 		(fields_autoplaced yes)
 		(effects
@@
 		)
 		(property "Intersheetrefs" "${INTERSHEET_REFS}"
-			(at 248.9476 83.82 0)
+			(at 248.9476 85.09 0)
 			(effects
 				(font
@@
 	(global_label "OUT_ENABLE"
 		(shape input)
-		(at 44.45 246.38 180)
+		(at 27.94 228.6 180)
 		(fields_autoplaced yes)
 		(effects
@@
 		)
 		(property "Intersheetrefs" "${INTERSHEET_REFS}"
-			(at 30.5076 246.38 0)
+			(at 13.9976 228.6 0)
 			(effects
 				(font
@@
 	(global_label "GND"
 		(shape input)
+		(at 29.21 236.22 270)
+		(fields_autoplaced yes)
+		(effects
+			(font
+				(size 1.27 1.27)
+			)
+			(justify right)
+		)
+		(property "Intersheetrefs" "${INTERSHEET_REFS}"
+			(at 1.27 100.33 0)
+			(effects
+				(font
+					(size 1.27 1.27)
+				)
+				(hide yes)
+			)
+		)
+	)
+	(global_label "GND"
+		(shape input)
 		(at 72.39 124.46 270)
 		(fields_autoplaced yes)
@@
 	(symbol
 		(lib_id "Device:R")
+		(at 29.21 232.41 180)
+		(unit 1)
+		(exclude_from_sim no)
+		(in_bom yes)
+		(on_board yes)
+		(dnp no)
+		(property "Reference" "R59"
+			(at 26.67 232.41 90)
+			(effects
+				(font
+					(size 1.27 1.27)
+				)
+			)
+		)
+		(property "Value" "10kΩ"
+			(at 29.464 232.41 90)
+			(effects
+				(font
+					(size 1.27 1.27)
+				)
+			)
+		)
+		(property "Footprint" "Resistor_SMD:R_0603_1608Metric_Pad0.98x0.95mm_HandSolder"
+			(at 30.988 232.41 90)
+			(effects
+				(font
+					(size 1.27 1.27)
+				)
+				(hide yes)
+			)
+		)
+		(property "Datasheet" "~"
+			(at 29.21 232.41 0)
+			(effects
+				(font
+					(size 1.27 1.27)
+				)
+				(hide yes)
+			)
+		)
+		(property "Description" "Resistor"
+			(at 29.21 232.41 0)
+			(effects
+				(font
+					(size 1.27 1.27)
+				)
+				(hide yes)
+			)
+		)
+		(property "JLCPCB" "C25804"
+			(at 29.21 232.41 90)
+			(effects
+				(font
+					(size 1.27 1.27)
+				)
+				(hide yes)
+			)
+		)
+		(property "LCSC" "C25804"
+			(at 29.21 232.41 0)
+			(effects
+				(font
+					(size 1.27 1.27)
+				)
+				(hide yes)
+			)
+		)
+		(property "Field4" ""
+			(at 29.21 232.41 0)
+			(effects
+				(font
+					(size 1.27 1.27)
+				)
+				(hide yes)
+			)
+		)
+		(pin "1"
+		)
+		(pin "2"
+		)
+		(instances
+			(project "hamodule"
+				(path "/e5217a0c-7f55-4c30-adda-7f8d95709d1b"
+					(reference "R59")
+					(unit 1)
+				)
+			)
+		)
+	)
+	(symbol
+		(lib_id "Device:R")
 		(at 228.6 58.42 270)
 		(unit 1)
@@
 		(on_board yes)
 		(dnp no)
-		(fields_autoplaced yes)
 		(property "Reference" "#FLG01"
 			(at 59.69 60.325 0)
@@
 		)
 		(property "Value" "PWR_FLAG"
-			(at 59.69 57.15 0)
+			(at 59.69 63.754 0)
 			(effects
 				(font
 					(size 1.27 1.27)
 				)
+				(hide yes)
 			)
 		)
@@
 			)
 		)
+		(property "PcbText" ""
+			(at 59.69 62.23 0)
+			(effects
+				(font
+					(size 1.27 1.27)
+				)
+			)
+		)
 		(pin "1"
 		)
@@
 	)
 	(symbol
-		(lib_id "Jumper:SolderJumper_2_Bridged")
+		(lib_id "Jumper:SolderJumper_2_Open")
 		(at 265.43 78.74 270)
 		(unit 1)
@@
 			)
 		)
-		(property "Footprint" "Jumper:SolderJumper-2_P1.3mm_Bridged2Bar_RoundedPad1.0x1.5mm"
+		(property "Footprint" "Jumper:SolderJumper-2_P1.3mm_Open_RoundedPad1.0x1.5mm"
 			(at 265.43 78.74 0)
 			(effects
@@
 			)
 		)
-		(property "Description" "Solder Jumper, 2-pole, closed/bridged"
+		(property "Description" "Solder Jumper, 2-pole, open"
 			(at 265.43 78.74 0)
 			(effects
@@
 	)
 	(symbol
-		(lib_id "Jumper:SolderJumper_2_Bridged")
+		(lib_id "Jumper:SolderJumper_2_Open")
 		(at 234.95 133.35 270)
 		(unit 1)
@@
 			)
 		)
-		(property "Footprint" "Jumper:SolderJumper-2_P1.3mm_Bridged2Bar_RoundedPad1.0x1.5mm"
+		(property "Footprint" "Jumper:SolderJumper-2_P1.3mm_Open_RoundedPad1.0x1.5mm"
 			(at 234.95 133.35 0)
 			(effects
@@
 			)
 		)
-		(property "Description" "Solder Jumper, 2-pole, closed/bridged"
+		(property "Description" "Solder Jumper, 2-pole, open"
 			(at 234.95 133.35 0)
 			(effects
@@
 		(dnp no)
 		(property "Reference" "U2"
-			(at 80.772 126.238 0)
+			(at 84.328 126.492 0)
 			(effects
 				(font
@@
 		)
 		(property "Value" "USBLC6-2SC6"
-			(at 92.202 128.27 0)
+			(at 95.504 128.524 0)
 			(effects
 				(font
@@
 	(symbol
 		(lib_id "Device:R")
-		(at 257.81 78.74 90)
+		(at 256.54 78.74 90)
 		(unit 1)
 		(exclude_from_sim no)
@@
 		(dnp no)
 		(property "Reference" "R61"
-			(at 257.81 76.454 90)
+			(at 256.54 76.454 90)
 			(effects
 				(font
@@
 		)
 		(property "Value" "10kΩ"
-			(at 257.81 78.74 90)
+			(at 256.54 78.74 90)
 			(effects
 				(font
@@
 		)
 		(property "Footprint" "Resistor_SMD:R_0603_1608Metric_Pad0.98x0.95mm_HandSolder"
-			(at 257.81 80.518 90)
+			(at 256.54 80.518 90)
 			(effects
 				(font
@@
 		)
 		(property "Datasheet" "~"
-			(at 257.81 78.74 0)
+			(at 256.54 78.74 0)
 			(effects
 				(font
@@
 		)
 		(property "Description" "Resistor"
-			(at 257.81 78.74 0)
+			(at 256.54 78.74 0)
 			(effects
 				(font
@@
 		)
 		(property "JLCPCB" "C25804"
-			(at 257.81 78.74 90)
+			(at 256.54 78.74 90)
 			(effects
 				(font
@@
 		)
 		(property "LCSC" "C25804"
-			(at 257.81 78.74 0)
+			(at 256.54 78.74 0)
 			(effects
 				(font
@@
 		)
 		(property "Field4" ""
-			(at 257.81 78.74 0)
+			(at 256.54 78.74 0)
 			(effects
 				(font
