File: PCB/schematics-v28.2/kicad/hamodule.kicad_pcb (KiCad board)
At the start: 4 copper layers, 78.4 x 84.3 mm, 104 parts, among them J10 Serial, J11 USB_C_Receptacle_USB2.0, J12 2604-1104, J13 EspSense, J14 I2C, J15 I2C, J2 2604-1102, J3 I2C, J4 13|12, J5 9|3|16, J7 Current Jumper, J8 EspRelays, J9 2604-1104, K1 AQG12205, K2 AQG12205, K3 AQG12205, K4 AQG12205, SW1 Switch, SW2 Switch, SW3 USB | PS, U1 LD1117AV33, U2 ESP32-S3-WROOM-2, U3 ULN2003A, U4 USBLC6-2SC6, U5 LDA210-PDIP, U6 LDA210-PDIP, U7 SHT4x

Commit message: v28
Parts:
- removed U3: ULN2003A, Package_SO:SOIC-16_3.9x9.9mm_P1.27mm
- added D8: LED, LED_SMD:LED_0805_2012Metric_Pad1.15x1.40mm_HandSolder, F.Cu at (40.2, 102.9)
- added R26: 100Ω, Resistor_SMD:R_0805_2012Metric_Pad1.20x1.40mm_HandSolder, F.Cu at (40.2, 99.2)
- added U11: ULN2803A, Package_SO:SOIC-18W_7.5x11.6mm_P1.27mm, F.Cu at (84.4, 85.3)
- J5: value 9|3|16 -> 9|3|46
- SW3: value USB | PS -> USB|PS
- moved G2 50.3 mm to (129.2, 93.8)
- moved D1 34.8 mm to (42.2, 102.9), turned to 90 degrees
- moved R2 31.0 mm to (42.1, 99.2), turned to 90 degrees
- moved G4 16.6 mm to (71.9, 98.2), turned to -90 degrees
- moved SW1 15.0 mm to (69.7, 83.8)
- moved J14 6.38 mm to (62.4, 108.5)
- moved J8 5.34 mm to (74.7, 81.5), turned to 0 degrees
- moved J5 5.28 mm to (81.9, 94.9), turned to 90 degrees
- moved J15 4.43 mm to (57.4, 111.0), turned to 180 degrees
- moved C14 3.61 mm to (86.9, 75.5), turned to -90 degrees
- moved D4 1.69 mm to (73.5, 96.5)
- moved D5 1.69 mm to (75.1, 96.5)
- moved D6 1.69 mm to (76.8, 96.5)
- moved D7 1.69 mm to (78.5, 96.5)
- moved R23 1.69 mm to (73.5, 93.1)
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- renumbered Rr1 to R27
Connections:
- J5 pad 3: GPIO16 -> GPIO46
- U2 pad 10: EspRel4 -> EspRel2
- U2 pad 12: EspRel2 -> EspRel4
- U2 pad 15: GPIO3 -> EspRel1
- U2 pad 16: EspRel1 -> GPIO46
- U2 pad 9: GPIO16 -> GPIO3
Routing:
- net 3.3V+: track 115.3 -> 163.7 mm
- net GND: track 164.8 -> 128.4 mm, vias 50 -> 49
- net 5V+: track 85.3 -> 112.3 mm
- net GPIO3: track 3.54 -> 17.6 mm, vias 0 -> 1
- net EspRel1: track 37.7 -> 23.8 mm
- net GPIO16: track 13.7 -> 0.00 mm, vias 2 -> 0
- net EspRel4: track 29.5 -> 41.9 mm
- net EN: track 37.9 -> 49.7 mm, vias 3 -> 2
- net EspRel3: track 31.0 -> 38.4 mm
- net GPIO9: track 3.54 -> 8.84 mm
- net GPIO46: track 0.00 -> 3.23 mm
- net EspRel2: track 33.5 -> 36.3 mm
- net Net-(D8-A): track 0.00 -> 1.72 mm
- net Net-(D1-A): track 2.92 -> 1.75 mm
- net Net-(U11-O5): track 16.3 -> 17.4 mm

Commit message: [v28] Adding stitching vias, and vias where USB change layer.
Parts:
- U7: footprint sht40:XDCR_SHT40-AD1B-R2 -> Sensor_Humidity:Sensirion_DFN-4_1.5x1.5mm_P0.8mm_SHT4x_NoCentralPad
- moved G2 85.6 mm to (44.1, 103.1)
- moved G4 2.00 mm to (69.9, 98.2)
Routing:
- net GND: track 128.4 -> 129.3 mm, vias 49 -> 72
Other:
- board text removed: "JLCJLCJLCJLC"

Commit message: [v28] Updated part numbers from JLCPCB and version in the silkscreen
Parts:
- C10, C11, C20, C6, C7: value NC -> 22uF
- C2: value NC -> 100uF
- C21, C8: value 10uF -> 100uF
- J14, J15, J3: value I2C -> ~
Routing:
- net EspRel3: track 38.4 -> 40.9 mm
- net EspRel2: track 36.3 -> 38.8 mm
- net EspRel4: track 41.9 -> 44.0 mm
- net EN: track 49.7 -> 50.7 mm
- net GND: vias 72 -> 70
Other:
- board text added: "V.20260701.28.2"
- board text removed: "V.20230201.22"
